Commit message: some changes on control and urdf

File: PARAM/lbr_description/urdf/Grieel/grieel_gazebo_phisics.xacro (robot description, xacro)
@@ -20,6 +20,6 @@
         <xacro:unless value="$(arg wheel_mode)">
             <gazebo reference="${prefix}_gripper_Link">
-                <mu1>1.2</mu1>
-                <mu2>1.2</mu2>
+                <mu1>0.6</mu1>
+                <mu2>0.6</mu2>
                 <kp>1000000</kp>
                 <kd>1.0</kd>

File: PARAM/lbr_description/urdf/Grieel/grieel_gripper_description.xacro (robot description, xacro)
@@ -243,5 +243,5 @@
       effort="0.0"
       velocity="0.0" />
-    <dynamics damping="0.1" friction="1.5"/>
+    <dynamics damping="0.1" friction="0.4"/>
   </joint>
     <!-- Gazebo plugin for contact sensor, collision name like that because of parsing errors in the urdf  -->

File: PARAM/lbr_description/urdf/Grieel/lbr_ros2_control.xacro (robot description, xacro)
@@ -12,6 +12,8 @@
         </command_interface>
         <command_interface name="velocity">
-          <param name="min">-2.8</param>
-          <param name="max">2.8</param>
+          <!-- <param name="min">-2.8</param>
+          <param name="max">2.8</param> -->
+          <param name="min">-10</param>
+          <param name="max">10</param>
         </command_interface>
         <command_interface name="effort">
@@ -26,9 +28,9 @@
         <state_interface name="velocity"/>
         <state_interface name="effort"/>
-        <transmission name="${prefix}_B2C_transmission">
+        <!-- <transmission name="${prefix}_B2C_transmission">
           <plugin>transmission_interface/SimpleTransmission</plugin>
           <param name="joint_to_actuator">272.5</param>
           <hardwareInterface>EffortJointInterface</hardwareInterface>
-        </transmission>
+        </transmission> -->
       </joint>
       <joint name="${prefix}_C2F">
@@ -38,6 +40,8 @@
         </command_interface>
         <command_interface name="velocity">
-          <param name="min">-2.8</param>
-          <param name="max">2.8</param>
+          <!-- <param name="min">-2.8</param>
+          <param name="max">2.8</param> -->
+          <param name="min">-10</param>
+          <param name="max">10</param>
         </command_interface>
         <command_interface name="effort">
@@ -52,9 +56,9 @@
         <state_interface name="velocity"/>
         <state_interface name="effort"/>
-        <transmission name="${prefix}_C2F_transmission">
+        <!-- <transmission name="${prefix}_C2F_transmission">
           <plugin>transmission_interface/SimpleTransmission</plugin>
           <param name="joint_to_actuator">272.5</param>
           <hardwareInterface>EffortJointInterface</hardwareInterface>
-        </transmission>
+        </transmission> -->
       </joint>
       <joint name="${prefix}_F2T">
@@ -64,6 +68,8 @@
         </command_interface>
         <command_interface name="velocity">
-          <param name="min">-4</param>
-          <param name="max">4</param>
+          <!-- <param name="min">-4</param>
+          <param name="max">4</param> -->
+          <param name="min">-10</param>
+          <param name="max">10</param>
         </command_interface>
         <command_interface name="effort">
@@ -78,9 +84,9 @@
         <state_interface name="velocity"/>
         <state_interface name="effort"/>
-        <transmission name="${prefix}_F2T_transmission">
+        <!-- <transmission name="${prefix}_F2T_transmission">
           <plugin>transmission_interface/SimpleTransmission</plugin>
           <param name="joint_to_actuator">353.5</param>
           <hardwareInterface>EffortJointInterface</hardwareInterface>
-        </transmission>
+        </transmission> -->
       </joint>
       <joint name="${prefix}_T2E">
@@ -90,6 +96,8 @@
         </command_interface>
         <command_interface name="velocity">
-          <param name="min">-4</param>
-          <param name="max">4</param>
+          <!-- <param name="min">-4</param>
+          <param name="max">4</param> -->
+          <param name="min">-10</param>
+          <param name="max">10</param>
         </command_interface>
         <command_interface name="effort">
@@ -104,9 +112,9 @@
         <state_interface name="velocity"/>
         <state_interface name="effort"/>
-        <transmission name="${prefix}_T2E_transmission">
+        <!-- <transmission name="${prefix}_T2E_transmission">
           <plugin>transmission_interface/SimpleTransmission</plugin>
           <param name="joint_to_actuator">353.5</param>
           <hardwareInterface>EffortJointInterface</hardwareInterface>
-        </transmission>
+        </transmission> -->
       </joint>
       <joint name="${prefix}_wristH">
@@ -116,6 +124,8 @@
         </command_interface>
         <command_interface name="velocity">
-          <param name="min">-5</param>
-          <param name="max">5</param>
+          <!-- <param name="min">-5</param>
+          <param name="max">5</param> -->
+          <param name="min">-10</param>
+          <param name="max">10</param>
         </command_interface>
         <command_interface name="effort">
@@ -135,9 +145,9 @@
         <state_interface name="velocity"/>
         <state_interface name="effort"/>
-        <transmission name="${prefix}_wristH_transmission">
+        <!-- <transmission name="${prefix}_wristH_transmission">
           <plugin>transmission_interface/SimpleTransmission</plugin>
           <param name="joint_to_actuator">257.4</param>
           <hardwareInterface>EffortJointInterface</hardwareInterface>
-        </transmission>
+        </transmission> -->
       </joint>
       <joint name="${prefix}_wristV">
@@ -147,6 +157,8 @@
         </command_interface>
         <command_interface name="velocity">
-          <param name="min">-5</param>
-          <param name="max">5</param>
+          <!-- <param name="min">-5</param>
+          <param name="max">5</param> -->
+          <param name="min">-10</param>
+          <param name="max">10</param>
         </command_interface>
         <command_interface name="effort">
@@ -166,9 +178,9 @@
         <state_interface name="velocity"/>
         <state_interface name="effort"/>
-        <transmission name="${prefix}_wristV_transmission">
+        <!-- <transmission name="${prefix}_wristV_transmission">
           <plugin>transmission_interface/SimpleTransmission</plugin>
           <param name="joint_to_actuator">257.4</param>
           <hardwareInterface>EffortJointInterface</hardwareInterface>
-        </transmission>
+        </transmission> -->
       </joint>
       <joint name="${prefix}_driving">
@@ -178,6 +190,8 @@
         </command_interface>
         <command_interface name="velocity">
-          <param name="min">-4</param>
-          <param name="max">4</param>
+          <!-- <param name="min">-4</param>
+          <param name="max">4</param> -->
+          <param name="min">-10</param>
+          <param name="max">10</param>
         </command_interface>
         <command_interface name="effort">
@@ -197,9 +211,9 @@
         <state_interface name="velocity"/>
         <state_interface name="effort"/>
-        <transmission name="${prefix}_driving_transmission">
+        <!-- <transmission name="${prefix}_driving_transmission">
           <plugin>transmission_interface/SimpleTransmission</plugin>
           <param name="joint_to_actuator">353.4</param>
           <hardwareInterface>EffortJointInterface</hardwareInterface>
-        </transmission>
+        </transmission> -->
       </joint>
     </ros2_control>

Commit message: wheel driving working

File: PARAM/lbr_description/urdf/Grieel/grieel_gazebo_phisics.xacro (robot description, xacro)
@@ -12,6 +12,6 @@
         <xacro:if value="$(arg wheel_mode)">
             <gazebo reference="${prefix}_wheel_Link">
-                <mu1>1.5</mu1>
-                <mu2>2.5</mu2>
+                <mu1>2.5</mu1>
+                <mu2>5.0</mu2>
                 <kp>1000000</kp>
                 <kd>1.0</kd>

File: PARAM/lbr_description/urdf/Grieel/grieel_wheel_description.xacro (robot description, xacro)
@@ -242,4 +242,7 @@
     <axis
       xyz="1 0 0" />
+    <limit
+      effort="10"
+      velocity="5" />
     <dynamics damping="0.1" friction="0.4"/>
   </joint>
