Commit message: Ellipsoid visualization in Rviz

File: PARAM/lbr_description/urdf/Grieel/grieel_gripper_description.xacro (robot description, xacro)
@@ -244,4 +244,16 @@
       velocity="0.0" />
     <dynamics damping="0.1" friction="0.4"/>
+  </joint>
+  <link name="${prefix}_end_effector_DH_Link"/>
+  <joint
+    name="${prefix}_end_effector_DH"
+    type="fixed">
+    <origin
+      xyz="0.0 0 0.0"
+      rpy="-3.1416 -1.5708  0" />
+    <parent
+      link="${prefix}_gripper_Link" />
+    <child
+      link="${prefix}_end_effector_DH_Link" />
   </joint>
     <!-- Gazebo plugin for contact sensor, collision name like that because of parsing errors in the urdf  -->

Commit message: make contact works, WIP

File: PARAM/lbr_description/urdf/Grieel/grieel_gripper_description.xacro (robot description, xacro)
@@ -257,23 +257,30 @@
       link="${prefix}_end_effector_DH_Link" />
   </joint>
-    <!-- Gazebo plugin for contact sensor, collision name like that because of parsing errors in the urdf  -->
+  <link name="${prefix}_gripper_end"/>
+  <joint
+    name="${prefix}_gripper_Root2End"
+    type="fixed">
+    <origin
+      xyz="0.0975 0 0.0"
+      rpy="0 1.5708  0" />
+    <parent
+      link="${prefix}_gripper_Link" />
+    <child
+      link="${prefix}_gripper_end" />
+  </joint>
+    <!-- Gazebo plugin for contact sensor -->
   <!-- <gazebo reference="${prefix}_gripper_Link">
-    <plugin filename="gz-sim-contact-system" name="gz::sim::systems::Contact">
-          <target>ground_plane</target>
-          <time>0.001</time>
-          <enabled>true</enabled>
-          <namespace>${prefix}</namespace>
-    </plugin>
     <sensor name="sensor_contact" type="contact">
         <contact>
-            <collision>${prefix}_gripper_Link_collision</collision>
+            <collision>${prefix}_gripper_Link_collision_collision</collision>
         </contact>
-        <always_on>1</always_on>
-        <update_rate>1000</update_rate>
     </sensor>
-    <plugin filename="gz-sim-touchplugin-system" name="gz::sim::systems::TouchPlugin">
-        <target>LIMBERO/link/${prefix}_gripper_Link</target>
+  </gazebo>
+  <gazebo>
+    <plugin filename="gz-sim-touchplugin-system"
+                name="gz::sim::systems::TouchPlugin">
+        <target>ground_plane</target>
         <namespace>${prefix}</namespace>
-        <time>0.001</time>
+        <time>0.01</time>
         <enabled>true</enabled>
     </plugin>

File: PARAM/lbr_description/urdf/Grieel/lbr_grieel_transmission.xacro (robot description, xacro)
@@ -9,9 +9,9 @@
         <type>transmission_interface/SimpleTransmission</type>
           <joint name="${prefix}_B2C">
-            <hardwareInterface>EffortJointInterface</hardwareInterface>
+            <hardwareInterface>hardware_interface/EffortJointInterface</hardwareInterface>
           </joint>
           <actuator name="${prefix}_Dynamixel_B2C">
             <mechanicalReduction>272.5</mechanicalReduction>
-            <hardwareInterface>EffortJointInterface</hardwareInterface>
+            <hardwareInterface>hardware_interface/EffortJointInterface</hardwareInterface>
           </actuator>
       </transmission>
@@ -19,8 +19,8 @@
         <type>transmission_interface/SimpleTransmission</type>
           <joint name="${prefix}_C2F">
-            <hardwareInterface>EffortJointInterface</hardwareInterface>
+            <hardwareInterface>hardware_interface/EffortJointInterface</hardwareInterface>
           </joint>
           <actuator name="${prefix}_Dynamixel_C2F">
-            <hardwareInterface>EffortJointInterface</hardwareInterface>
+            <hardwareInterface>hardware_interface/EffortJointInterface</hardwareInterface>
             <mechanicalReduction>272.5</mechanicalReduction>
           </actuator>
@@ -29,9 +29,9 @@
         <type>transmission_interface/SimpleTransmission</type>
           <joint name="${prefix}_F2T">
-            <hardwareInterface>EffortJointInterface</hardwareInterface>
+            <hardwareInterface>hardware_interface/EffortJointInterface</hardwareInterface>
           </joint>
           <actuator name="${prefix}_Dynamixel_F2T">
             <mechanicalReduction>353.5</mechanicalReduction>
-            <hardwareInterface>EffortJointInterface</hardwareInterface>
+            <hardwareInterface>hardware_interface/EffortJointInterface</hardwareInterface>
           </actuator>
       </transmission>
@@ -39,9 +39,9 @@
         <type>transmission_interface/SimpleTransmission</type>
           <joint name="${prefix}_T2E">
-            <hardwareInterface>EffortJointInterface</hardwareInterface>
+            <hardwareInterface>hardware_interface/EffortJointInterface</hardwareInterface>
           </joint>
           <actuator name="${prefix}_Dynamixel_T2E">
             <mechanicalReduction>353.5</mechanicalReduction>
-            <hardwareInterface>EffortJointInterface</hardwareInterface>
+            <hardwareInterface>hardware_interface/EffortJointInterface</hardwareInterface>
           </actuator>
       </transmission>
@@ -49,9 +49,9 @@
         <type>transmission_interface/SimpleTransmission</type>
           <joint name="${prefix}_wristH">
-            <hardwareInterface>EffortJointInterface</hardwareInterface>
+            <hardwareInterface>hardware_interface/EffortJointInterface</hardwareInterface>
           </joint>
           <actuator name="${prefix}_Dynamixel_wristH">
             <mechanicalReduction>257.4</mechanicalReduction>
-            <hardwareInterface>EffortJointInterface</hardwareInterface>
+            <hardwareInterface>hardware_interface/EffortJointInterface</hardwareInterface>
           </actuator>
       </transmission>
@@ -59,9 +59,9 @@
         <type>transmission_interface/SimpleTransmission</type>
           <joint name="${prefix}_wristV">
-            <hardwareInterface>EffortJointInterface</hardwareInterface>
+            <hardwareInterface>hardware_interface/EffortJointInterface</hardwareInterface>
           </joint>
           <actuator name="${prefix}_Dynamixel_wristV">
             <mechanicalReduction>257.4</mechanicalReduction>
-            <hardwareInterface>EffortJointInterface</hardwareInterface>
+            <hardwareInterface>hardware_interface/EffortJointInterface</hardwareInterface>
           </actuator>
       </transmission>
@@ -69,9 +69,9 @@
         <type>transmission_interface/SimpleTransmission</type>
           <joint name="${prefix}_driving">
-            <hardwareInterface>EffortJointInterface</hardwareInterface>
+            <hardwareInterface>hardware_interface/EffortJointInterface</hardwareInterface>
           </joint>
           <actuator name="${prefix}_Dynamixel_driving">
             <mechanicalReduction>353.4</mechanicalReduction>
-            <hardwareInterface>EffortJointInterface</hardwareInterface>
+            <hardwareInterface>hardware_interface/EffortJointInterface</hardwareInterface>
           </actuator>
       </transmission>

Commit message: fake contact and wheel control

File: PARAM/lbr_description/urdf/Grieel/grieel_gripper_description.xacro (robot description, xacro)
@@ -270,5 +270,5 @@
   </joint>
     <!-- Gazebo plugin for contact sensor -->
-  <!-- <gazebo reference="${prefix}_gripper_Link">
+  <gazebo reference="${prefix}_gripper_Link">
     <sensor name="sensor_contact" type="contact">
         <contact>
@@ -282,8 +282,8 @@
         <target>ground_plane</target>
         <namespace>${prefix}</namespace>
-        <time>0.01</time>
+        <time>0.001</time>
         <enabled>true</enabled>
     </plugin>
-  </gazebo> -->
+  </gazebo>
   </xacro:macro>
 </robot>

File: PARAM/lbr_description/urdf/Grieel/grieel_wheel_description.xacro (robot description, xacro)
@@ -97,5 +97,5 @@
       <origin
         xyz="-0.014255 0 0"
-        rpy="0 0 0" />
+        rpy="-3.14159265358 0 0" />
       <geometry>
         <mesh
@@ -155,6 +155,6 @@
     <collision>
       <origin
-        xyz="-0.03325 0 0.024002"
-        rpy="0 0 0" />
+        xyz="0.024002  0 -0.03325 "
+        rpy="3.14159265358 -1.5708 0" />
       <geometry>
         <mesh
@@ -214,6 +214,6 @@
     <collision name="${prefix}_wheel_Link_collision">
       <origin
-        xyz="-0.079017 0 0.010898"
-        rpy="0 0 0" />
+        xyz="0.010898 0 -0.079017"
+        rpy="0 -1.5708 3.14159265358" />
       <geometry>
         <mesh
@@ -246,17 +246,18 @@
     <!-- Gazebo plugin for contact sensor, collision name like that because of parsing errors in the urdf  -->
   <gazebo reference="${prefix}_wheel_Link">
-    <sensor name="${prefix}_gripper_bumper_sensor" type="contact">
-      <always_on>true</always_on>
-      <update_rate>100</update_rate>
-      <contact>
-        <collision>${prefix}_wheel_Link_collision_collision</collision>
-      </contact>
-      <plugin name="${prefix}_gripper_bumper" filename="libgazebo_ros_bumper.so">
-        <ros>
-          <namespace>${prefix}</namespace>
-        </ros>
-        <frame_name>${prefix}_wheel_link</frame_name>
-      </plugin>
+    <sensor name="sensor_contact" type="contact">
+        <contact>
+            <collision>${prefix}_wheel_Link_collision_collision</collision>
+        </contact>
     </sensor>
+  </gazebo>
+  <gazebo>
+    <plugin filename="gz-sim-touchplugin-system"
+                name="gz::sim::systems::TouchPlugin">
+        <target>ground_plane</target>
+        <namespace>${prefix}</namespace>
+        <time>0.001</time>
+        <enabled>true</enabled>
+    </plugin>
   </gazebo>
   </xacro:macro>

Commit message: updates on GUI and mesh gripper

File: PARAM/lbr_description/urdf/Grieel/grieel_gripper_description.xacro (robot description, xacro)
@@ -203,6 +203,8 @@
         rpy="0 0 0" />
       <geometry>
-        <mesh
-          filename="file://$(find lbr_description)/meshes/Grieel_gripper_mode/gripper_Link.STL" />
+        <!-- <mesh
+          filename="file://$(find lbr_description)/meshes/Grieel_gripper_mode/gripper_Link.STL" /> -->
+        <mesh
+          filename="file://$(find lbr_description)/meshes/Grieel_gripper_mode/gripper_Link_NOSPIKES.stl" />
       </geometry>
       <material
@@ -220,6 +222,8 @@
         rpy="0 ${pi/2} 0" /> -->
       <geometry>
-        <mesh
-          filename="file://$(find lbr_description)/meshes/Grieel_gripper_mode/gripper_Link.STL" />
+        <!-- <mesh
+          filename="file://$(find lbr_description)/meshes/Grieel_gripper_mode/gripper_Link.STL" /> -->
+        <mesh
+          filename="file://$(find lbr_description)/meshes/Grieel_gripper_mode/gripper_Link_NOSPIKES.stl" />
           <!-- <cylinder radius="0.112" length="0.060"/> -->
       </geometry>

Commit message: GRIEEL Transformation simulation

File: PARAM/lbr_description/urdf/Grieel/grieel_gripper_description.xacro (robot description, xacro)
@@ -6,4 +6,5 @@
   name="assembled_gripper_mode" xmlns:xacro="http://ros.org/wiki/xacro">
   <xacro:macro name="grieel_gripper_macro" params="prefix parent">
+  <xacro:include filename="$(find lbr_description)/urdf/Grieel/grieel_gripper_splitted.xacro" />
     <joint
       name="${prefix}_E2grieel"
@@ -182,5 +183,5 @@
     <dynamics damping="0.1" friction="0.4"/>
   </joint>
-  <link
+  <!-- <link
     name="${prefix}_gripper_Link">
     <inertial>
@@ -203,6 +204,4 @@
         rpy="0 0 0" />
       <geometry>
-        <!-- <mesh
-          filename="file://$(find lbr_description)/meshes/Grieel_gripper_mode/gripper_Link.STL" /> -->
         <mesh
           filename="file://$(find lbr_description)/meshes/Grieel_gripper_mode/gripper_Link_NOSPIKES.stl" />
@@ -218,17 +217,12 @@
       xyz="0 0 0"
       rpy="0 0 0" />
-      <!-- <origin
-        xyz="0.05 0 0"
-        rpy="0 ${pi/2} 0" /> -->
-      <geometry>
-        <!-- <mesh
-          filename="file://$(find lbr_description)/meshes/Grieel_gripper_mode/gripper_Link.STL" /> -->
+      <geometry>
         <mesh
           filename="file://$(find lbr_description)/meshes/Grieel_gripper_mode/gripper_Link_NOSPIKES.stl" />
-          <!-- <cylinder radius="0.112" length="0.060"/> -->
-      </geometry>
-    </collision>
-  </link>
-  <joint
+      </geometry>
+    </collision>
+  </link> -->
+  <xacro:grieel_hand_macro prefix="${prefix}"/>
+  <!-- <joint
     name="${prefix}_driving"
     type="revolute">
@@ -272,7 +266,7 @@
     <child
       link="${prefix}_gripper_end" />
-  </joint>
+  </joint> -->
     <!-- Gazebo plugin for contact sensor -->
-  <gazebo reference="${prefix}_gripper_Link">
+  <!-- <gazebo reference="${prefix}_gripper_Link">
     <sensor name="sensor_contact" type="contact">
         <contact>
@@ -289,5 +283,5 @@
         <enabled>true</enabled>
     </plugin>
-  </gazebo>
+  </gazebo> -->
   </xacro:macro>
 </robot>

Commit message: new control stuff

File: PARAM/lbr_description/urdf/Grieel/grieel_gripper_description.xacro (robot description, xacro)
@@ -122,5 +122,5 @@
       effort="8.0"
       velocity="4.0" />
-    <dynamics damping="0.1" friction="0.4"/>
+    <dynamics damping="0.01" friction="0.1"/>
   </joint>
   <link
@@ -181,5 +181,5 @@
       effort="8.0"
       velocity="4.0" />
-    <dynamics damping="0.1" friction="0.4"/>
+    <dynamics damping="0.01" friction="0.1"/>
   </joint>
   <!-- <link

File: PARAM/lbr_description/urdf/Grieel/lbr_limb_description.xacro (robot description, xacro)
@@ -114,5 +114,5 @@
         effort="16.0"
         velocity="3.0" />
-      <dynamics damping="0.1" friction="0.4"/>
+      <dynamics damping="0.01" friction="0.1"/>
     </joint>
     <!-- <transmission name="${prefix}_B2C_transmission">
@@ -183,5 +183,5 @@
         effort="16.0"
         velocity="5.0" />
-      <dynamics damping="0.1" friction="0.4"/>
+      <dynamics damping="0.01" friction="0.1"/>
     </joint>
     <!-- <transmission name="${prefix}_C2F_transmission">
@@ -252,5 +252,5 @@
         effort="10.0"
         velocity="5.0" />
-      <dynamics damping="0.1" friction="0.4"/>
+      <dynamics damping="0.01" friction="0.1"/>
       <initial_position value="${pi/2}"/>
     </joint>
@@ -322,5 +322,5 @@
         effort="8.0"
         velocity="4.0" />
-      <dynamics damping="0.1" friction="0.4"/>
+      <dynamics damping="0.01" friction="0.1"/>
     </joint>
     <!-- <transmission name="${prefix}_T2E_transmission">
