Commit message: init branch

File: PARAM/lbr_description/urdf/Grieel/LIMBERO.xacro (robot description, xacro)
@@ -6,6 +6,4 @@
   <xacro:include filename="$(find lbr_description)/urdf/Grieel/grieel_joint_state.xacro" />
   <xacro:include filename="$(find lbr_description)/urdf/Grieel/grieel_gazebo_phisics.xacro" />
-  <xacro:include filename="$(find lbr_description)/urdf/Grieel/lbr_grieel_transmission.xacro" />
-  <xacro:include filename="$(find lbr_description)/urdf/Grieel/lidar.xacro" />
   <!-- Use macro to define base and four limbs -->
   <xacro:base_macro/>
@@ -43,8 +41,4 @@
   <xacro:joint_state_macro prefix="RH"/>
   <xacro:joint_state_macro prefix="RF"/>
-  <!-- <xacro:transmission_macro prefix="LF"/>
-  <xacro:transmission_macro prefix="LH"/>
-  <xacro:transmission_macro prefix="RH"/>
-  <xacro:transmission_macro prefix="RF"/> -->
   <xacro:gazebo_phisics_macro prefix="LF"/>
   <xacro:gazebo_phisics_macro prefix="LH"/>

File: PARAM/lbr_description/urdf/Grieel/grieel_gazebo_phisics.xacro (robot description, xacro)
@@ -20,6 +20,6 @@
         <xacro:unless value="$(arg wheel_mode)">
             <gazebo reference="${prefix}_gripper_Link">
-                <mu1>1.2</mu1>
-                <mu2>1.2</mu2>
+                <mu1>0.5</mu1>
+                <mu2>0.5</mu2>
                 <kp>1000000</kp>
                 <kd>1.0</kd>

File: PARAM/lbr_description/urdf/Grieel/grieel_gripper_description.xacro (robot description, xacro)
@@ -119,6 +119,6 @@
       lower="-3.14159265358"
       upper="3.14159265358"
-      effort="50"
-      velocity="10" />
+      effort="5"
+      velocity="5" />
     <dynamics damping="0.1" friction="0.4"/>
   </joint>
@@ -178,6 +178,6 @@
       lower="-0.78539816339"
       upper="1.57079632679"
-      effort="50"
-      velocity="10" />
+      effort="5"
+      velocity="5" />
     <dynamics damping="0.1" friction="0.4"/>
   </joint>
@@ -214,13 +214,9 @@
     <collision name="${prefix}_gripper_Link_collision">
       <origin
-      xyz="0 0 0"
-      rpy="0 0 0" />
-      <!-- <origin
-        xyz="0.05 0 0"
-        rpy="0 ${pi/2} 0" /> -->
+        xyz="0 0 0"
+        rpy="0 0 0" />
       <geometry>
         <mesh
           filename="file://$(find lbr_description)/meshes/Grieel_gripper_mode/gripper_Link.STL" />
-          <!-- <cylinder radius="0.112" length="0.060"/> -->
       </geometry>
     </collision>
@@ -228,5 +224,5 @@
   <joint
     name="${prefix}_driving"
-    type="revolute">
+    type="continuous">
     <origin
       xyz="0.0131 0 0.04576"
@@ -237,11 +233,6 @@
       link="${prefix}_gripper_Link" />
     <axis
-      xyz="1 0 0" />
-    <limit
-      lower="-0.0"
-      upper="0.0"
-      effort="0.0"
-      velocity="0.0" />
-    <dynamics damping="0.1" friction="1.5"/>
+      xyz="-1 0 0" />
+    <dynamics damping="0.1" friction="0.4"/>
   </joint>
     <!-- Gazebo plugin for contact sensor, collision name like that because of parsing errors in the urdf  -->
@@ -249,5 +240,5 @@
       <sensor name="${prefix}_gripper_bumper_sensor" type="contact">
         <always_on>true</always_on>
-        <update_rate>50</update_rate>
+        <update_rate>100</update_rate>
         <contact>
         <collision>${prefix}_gripper_Link_collision_collision</collision>

File: PARAM/lbr_description/urdf/Grieel/grieel_joint_state.xacro (robot description, xacro)
@@ -17,5 +17,5 @@
                 <remapping>~/out:=joint_states</remapping>
             </ros>
-            <update_rate>500</update_rate>
+            <update_rate>30</update_rate>
             <!-- <joint_name>${prefix}_E2grieel</joint_name> -->
             <joint_name>${prefix}_B2C</joint_name>

File: PARAM/lbr_description/urdf/Grieel/grieel_wheel_description.xacro (robot description, xacro)
@@ -241,5 +241,5 @@
       link="${prefix}_wheel_Link" />
     <axis
-      xyz="1 0 0" />
+      xyz="-1 0 0" />
     <dynamics damping="0.1" friction="0.4"/>
   </joint>

File: PARAM/lbr_description/urdf/Grieel/lbr_limb_description.xacro (robot description, xacro)
@@ -112,18 +112,8 @@
         lower="-3.14"
         upper="3.14"
-        effort="50"
-        velocity="10" />
-      <dynamics damping="0.1" friction="0.4"/>
-    </joint>
-    <!-- <transmission name="${prefix}_B2C_transmission">
-      <type>transmission_interface/SimpleTransmission</type>
-        <joint name="${prefix}_B2C">
-          <hardwareInterface>EffortJointInterface</hardwareInterface>
-        </joint>
-        <actuator name="${prefix}_Dynamixel_B2C">
-          <mechanicalReduction>272.5</mechanicalReduction>
-          <hardwareInterface>EffortJointInterface</hardwareInterface>
-        </actuator>
-    </transmission> -->
+        effort="5"
+        velocity="5" />
+      <dynamics damping="0.1" friction="0.4"/>
+    </joint>
     <link
       name="${prefix}_femur">
@@ -181,18 +171,8 @@
         lower="-3.14"
         upper="3.14"
-        effort="50"
-        velocity="10" />
-      <dynamics damping="0.1" friction="0.4"/>
-    </joint>
-    <!-- <transmission name="${prefix}_C2F_transmission">
-      <type>transmission_interface/SimpleTransmission</type>
-        <joint name="${prefix}_C2F">
-          <hardwareInterface>EffortJointInterface</hardwareInterface>
-        </joint>
-        <actuator name="${prefix}_Dynamixel_C2F">
-          <hardwareInterface>EffortJointInterface</hardwareInterface>
-          <mechanicalReduction>272.5</mechanicalReduction>
-        </actuator>
-    </transmission> -->
+        effort="5"
+        velocity="5" />
+      <dynamics damping="0.1" friction="0.4"/>
+    </joint>
     <link
       name="${prefix}_tibia">
@@ -250,18 +230,8 @@
         lower="-3.14"
         upper="3.14"
-        effort="50"
-        velocity="10" />
-      <dynamics damping="0.1" friction="0.4"/>
-    </joint>
-    <!-- <transmission name="${prefix}_F2T_transmission">
-      <type>transmission_interface/SimpleTransmission</type>
-        <joint name="${prefix}_F2T">
-          <hardwareInterface>EffortJointInterface</hardwareInterface>
-        </joint>
-        <actuator name="${prefix}_Dynamixel_F2T">
-          <mechanicalReduction>353.5</mechanicalReduction>
-          <hardwareInterface>EffortJointInterface</hardwareInterface>
-        </actuator>
-    </transmission> -->
+        effort="5"
+        velocity="5" />
+      <dynamics damping="0.1" friction="0.4"/>
+    </joint>
     <link
       name="${prefix}_limb_end">
@@ -319,18 +289,8 @@
         lower="-3.14"
         upper="3.14"
-        effort="50"
-        velocity="10" />
-      <dynamics damping="0.1" friction="0.4"/>
-    </joint>
-    <!-- <transmission name="${prefix}_T2E_transmission">
-      <type>transmission_interface/SimpleTransmission</type>
-        <joint name="${prefix}_T2E">
-          <hardwareInterface>EffortJointInterface</hardwareInterface>
-        </joint>
-        <actuator name="${prefix}_Dynamixel_T2E">
-          <mechanicalReduction>353.5</mechanicalReduction>
-          <hardwareInterface>EffortJointInterface</hardwareInterface>
-        </actuator>
-    </transmission> -->
+        effort="5"
+        velocity="5" />
+      <dynamics damping="0.1" friction="0.4"/>
+    </joint>
   </xacro:macro>
 </robot>

File: PARAM/lbr_description/urdf/Grieel/lbr_ros2_control.xacro (robot description, xacro)
@@ -12,12 +12,10 @@
         </command_interface>
         <command_interface name="velocity">
-          <param name="min">-2.8</param>
-          <param name="max">2.8</param>
+          <param name="min">-0.5</param>
+          <param name="max">0.5</param>
         </command_interface>
         <command_interface name="effort">
-          <!-- <param name="min">-8</param>
-          <param name="max">8</param> -->
-          <param name="min">-50</param>
-          <param name="max">50</param>
+          <param name="min">-10</param>
+          <param name="max">10</param>
         </command_interface>
         <state_interface name="position">  <!-- Set initial joint position -->
@@ -25,10 +23,4 @@
         </state_interface>
         <state_interface name="velocity"/>
-        <state_interface name="effort"/>
-        <transmission name="${prefix}_B2C_transmission">
-          <plugin>transmission_interface/SimpleTransmission</plugin>
-          <param name="joint_to_actuator">272.5</param>
-          <hardwareInterface>EffortJointInterface</hardwareInterface>
-        </transmission>
       </joint>
       <joint name="${prefix}_C2F">
@@ -38,12 +30,10 @@
         </command_interface>
         <command_interface name="velocity">
-          <param name="min">-2.8</param>
-          <param name="max">2.8</param>
+          <param name="min">-0.5</param>
+          <param name="max">0.5</param>
         </command_interface>
         <command_interface name="effort">
-          <!-- <param name="min">-8</param>
-          <param name="max">8</param> -->
-          <param name="min">-50</param>
-          <param name="max">50</param>
+          <param name="min">-10</param>
+          <param name="max">10</param>
         </command_interface>
         <state_interface name="position">
@@ -51,10 +41,4 @@
         </state_interface>
         <state_interface name="velocity"/>
-        <state_interface name="effort"/>
-        <transmission name="${prefix}_C2F_transmission">
-          <plugin>transmission_interface/SimpleTransmission</plugin>
-          <param name="joint_to_actuator">272.5</param>
-          <hardwareInterface>EffortJointInterface</hardwareInterface>
-        </transmission>
       </joint>
       <joint name="${prefix}_F2T">
@@ -64,12 +48,10 @@
         </command_interface>
         <command_interface name="velocity">
-          <param name="min">-4</param>
-          <param name="max">4</param>
+          <param name="min">-0.5</param>
+          <param name="max">0.5</param>
         </command_interface>
         <command_interface name="effort">
-          <!-- <param name="min">-3.4</param>
-          <param name="max">3.4</param> -->
-          <param name="min">-50</param>
-          <param name="max">50</param>
+          <param name="min">-10</param>
+          <param name="max">10</param>
         </command_interface>
         <state_interface name="position">
@@ -77,25 +59,17 @@
         </state_interface>
         <state_interface name="velocity"/>
-        <state_interface name="effort"/>
-        <transmission name="${prefix}_F2T_transmission">
-          <plugin>transmission_interface/SimpleTransmission</plugin>
-          <param name="joint_to_actuator">353.5</param>
-          <hardwareInterface>EffortJointInterface</hardwareInterface>
-        </transmission>
       </joint>
       <joint name="${prefix}_T2E">
         <command_interface name="position">
-          <param name="min">-100</param>
-          <param name="max">100</param>
+          <param name="min">-10</param>
+          <param name="max">10</param>
         </command_interface>
         <command_interface name="velocity">
-          <param name="min">-4</param>
-          <param name="max">4</param>
+          <param name="min">-0.5</param>
+          <param name="max">0.5</param>
         </command_interface>
         <command_interface name="effort">
-          <!-- <param name="min">-3.4</param>
-          <param name="max">3.4</param> -->
-          <param name="min">-50</param>
-          <param name="max">50</param>
+          <param name="min">-10</param>
+          <param name="max">10</param>
         </command_interface>
         <state_interface name="position">
@@ -103,10 +77,4 @@
         </state_interface>
         <state_interface name="velocity"/>
-        <state_interface name="effort"/>
-        <transmission name="${prefix}_T2E_transmission">
-          <plugin>transmission_interface/SimpleTransmission</plugin>
-          <param name="joint_to_actuator">353.5</param>
-          <hardwareInterface>EffortJointInterface</hardwareInterface>
-        </transmission>
       </joint>
       <joint name="${prefix}_wristH">
@@ -116,12 +84,10 @@
         </command_interface>
         <command_interface name="velocity">
-          <param name="min">-5</param>
-          <param name="max">5</param>
+          <param name="min">-0.5</param>
+          <param name="max">0.5</param>
         </command_interface>
         <command_interface name="effort">
-          <!-- <param name="min">-1.20</param>
-          <param name="max">1.20</param> -->
-          <param name="min">-50</param>
-          <param name="max">50</param>
+          <param name="min">-10</param>
+          <param name="max">10</param>
         </command_interface>
         <state_interface name="position">
@@ -134,10 +100,4 @@
         </state_interface>
         <state_interface name="velocity"/>
-        <state_interface name="effort"/>
-        <transmission name="${prefix}_wristH_transmission">
-          <plugin>transmission_interface/SimpleTransmission</plugin>
-          <param name="joint_to_actuator">257.4</param>
-          <hardwareInterface>EffortJointInterface</hardwareInterface>
-        </transmission>
       </joint>
       <joint name="${prefix}_wristV">
@@ -147,12 +107,10 @@
         </command_interface>
         <command_interface name="velocity">
-          <param name="min">-5</param>
-          <param name="max">5</param>
+          <param name="min">-0.5</param>
+          <param name="max">0.5</param>
         </command_interface>
         <command_interface name="effort">
-          <!-- <param name="min">-1.20</param>
-          <param name="max">1.20</param> -->
-          <param name="min">-50</param>
-          <param name="max">50</param>
+          <param name="min">-10</param>
+          <param name="max">10</param>
         </command_interface>
         <state_interface name="position">
@@ -165,10 +123,4 @@
         </state_interface>
         <state_interface name="velocity"/>
-        <state_interface name="effort"/>
-        <transmission name="${prefix}_wristV_transmission">
-          <plugin>transmission_interface/SimpleTransmission</plugin>
-          <param name="joint_to_actuator">257.4</param>
-          <hardwareInterface>EffortJointInterface</hardwareInterface>
-        </transmission>
       </joint>
       <joint name="${prefix}_driving">
@@ -178,12 +130,10 @@
         </command_interface>
         <command_interface name="velocity">
-          <param name="min">-4</param>
-          <param name="max">4</param>
+          <param name="min">-0.5</param>
+          <param name="max">0.5</param>
         </command_interface>
         <command_interface name="effort">
-          <!-- <param name="min">-3.4</param>
-          <param name="max">3.4</param> -->
-          <param name="min">-50</param>
-          <param name="max">50</param>
+          <param name="min">-10</param>
+          <param name="max">10</param>
         </command_interface>
         <state_interface name="position">
@@ -196,10 +146,4 @@
         </state_interface>
         <state_interface name="velocity"/>
-        <state_interface name="effort"/>
-        <transmission name="${prefix}_driving_transmission">
-          <plugin>transmission_interface/SimpleTransmission</plugin>
-          <param name="joint_to_actuator">353.4</param>
-          <hardwareInterface>EffortJointInterface</hardwareInterface>
-        </transmission>
       </joint>
     </ros2_control>

Commit message: update for migration

File: PARAM/lbr_description/urdf/Grieel/LIMBERO.xacro (robot description, xacro)
@@ -2,10 +2,11 @@
   <xacro:include filename="$(find lbr_description)/urdf/Grieel/lbr_base_description.xacro" />
   <xacro:include filename="$(find lbr_description)/urdf/Grieel/lbr_limb_description.xacro" />
-  <xacro:include filename="$(find lbr_description)/urdf/Grieel/lbr_gazebo.xacro" />
-  <xacro:include filename="$(find lbr_description)/urdf/Grieel/lbr_ros2_control.xacro" />
+  <!-- <xacro:include filename="$(find lbr_description)/urdf/Grieel/lbr_gazebo.xacro" /> -->
+  <!-- <xacro:include filename="$(find lbr_description)/urdf/Grieel/lbr_ros2_control.xacro" /> -->
   <xacro:include filename="$(find lbr_description)/urdf/Grieel/grieel_joint_state.xacro" />
+  <xacro:include filename="$(find lbr_description)/urdf/Grieel/lbr_grieel_joint_actuation.xacro" />
   <xacro:include filename="$(find lbr_description)/urdf/Grieel/grieel_gazebo_phisics.xacro" />
-  <xacro:include filename="$(find lbr_description)/urdf/Grieel/lbr_grieel_transmission.xacro" />
-  <xacro:include filename="$(find lbr_description)/urdf/Grieel/lidar.xacro" />
+  <!-- <xacro:include filename="$(find lbr_description)/urdf/Grieel/lbr_grieel_transmission.xacro" /> -->
+  <!-- <xacro:include filename="$(find lbr_description)/urdf/Grieel/lidar.xacro" /> -->
   <!-- Use macro to define base and four limbs -->
   <xacro:base_macro/>
@@ -22,8 +23,8 @@
     <xacro:grieel_wheel_macro prefix="RH" parent="RH"/>
     <xacro:grieel_wheel_macro prefix="RF" parent="RF"/>
-    <xacro:ros2_control_macro prefix="LF" wheel_mode= "true"/>
+    <!-- <xacro:ros2_control_macro prefix="LF" wheel_mode= "true"/>
     <xacro:ros2_control_macro prefix="LH" wheel_mode= "true"/>
     <xacro:ros2_control_macro prefix="RH" wheel_mode= "true"/>
-    <xacro:ros2_control_macro prefix="RF" wheel_mode= "true"/>
+    <xacro:ros2_control_macro prefix="RF" wheel_mode= "true"/> -->
   </xacro:if>
   <!-- Grieel gripper mode -->
@@ -34,8 +35,8 @@
     <xacro:grieel_gripper_macro prefix="RH" parent="RH"/>
     <xacro:grieel_gripper_macro prefix="RF" parent="RF"/>
-    <xacro:ros2_control_macro prefix="LF" wheel_mode= "false"/>
+    <!-- <xacro:ros2_control_macro prefix="LF" wheel_mode= "false"/>
     <xacro:ros2_control_macro prefix="LH" wheel_mode= "false"/>
     <xacro:ros2_control_macro prefix="RH" wheel_mode= "false"/>
-    <xacro:ros2_control_macro prefix="RF" wheel_mode= "false"/>
+    <xacro:ros2_control_macro prefix="RF" wheel_mode= "false"/> -->
   </xacro:unless>
   <xacro:joint_state_macro prefix="LF"/>
@@ -43,4 +44,8 @@
   <xacro:joint_state_macro prefix="RH"/>
   <xacro:joint_state_macro prefix="RF"/>
+  <xacro:joint_actuator_macro prefix="LF"/>
+  <xacro:joint_actuator_macro prefix="LH"/>
+  <xacro:joint_actuator_macro prefix="RH"/>
+  <xacro:joint_actuator_macro prefix="RF"/>
   <!-- <xacro:transmission_macro prefix="LF"/>
   <xacro:transmission_macro prefix="LH"/>

File: PARAM/lbr_description/urdf/Grieel/grieel_gripper_description.xacro (robot description, xacro)
@@ -258,19 +258,25 @@
   </joint>
     <!-- Gazebo plugin for contact sensor, collision name like that because of parsing errors in the urdf  -->
-    <gazebo reference="${prefix}_gripper_Link">
-      <sensor name="${prefix}_gripper_bumper_sensor" type="contact">
-        <always_on>true</always_on>
-        <update_rate>50</update_rate>
+  <!-- <gazebo reference="${prefix}_gripper_Link">
+    <plugin filename="gz-sim-contact-system" name="gz::sim::systems::Contact">
+          <target>ground_plane</target>
+          <time>0.001</time>
+          <enabled>true</enabled>
+          <namespace>${prefix}</namespace>
+    </plugin>
+    <sensor name="sensor_contact" type="contact">
         <contact>
-        <collision>${prefix}_gripper_Link_collision_collision</collision>
+            <collision>${prefix}_gripper_Link_collision</collision>
         </contact>
-        <plugin name="${prefix}_gripper_bumper" filename="libgazebo_ros_bumper.so">
-          <ros>
-            <namespace>${prefix}</namespace>
-          </ros>
-          <frame_name>${prefix}_gripper_link</frame_name>
-        </plugin>
-      </sensor>
-    </gazebo>
+        <always_on>1</always_on>
+        <update_rate>1000</update_rate>
+    </sensor>
+    <plugin filename="gz-sim-touchplugin-system" name="gz::sim::systems::TouchPlugin">
+        <target>LIMBERO/link/${prefix}_gripper_Link</target>
+        <namespace>${prefix}</namespace>
+        <time>0.001</time>
+        <enabled>true</enabled>
+    </plugin>
+  </gazebo> -->
   </xacro:macro>
 </robot>

File: PARAM/lbr_description/urdf/Grieel/grieel_joint_state.xacro (robot description, xacro)
@@ -12,11 +12,11 @@
             <!-- Gazebo plugin for joint state publisher  -->
         <gazebo>
-            <plugin name="${prefix}_joint_state" filename="libgazebo_ros_joint_state_publisher.so">
-            <ros>
+            <plugin name="gz::sim::systems::JointStatePublisher" filename="gz-sim-joint-state-publisher-system">
+            <!-- <ros>
                 <namespace>${prefix}</namespace>
                 <remapping>~/out:=joint_states</remapping>
-            </ros>
-            <update_rate>500</update_rate>
-            <!-- <joint_name>${prefix}_E2grieel</joint_name> -->
+            </ros> -->
+            <!-- <update_rate>500</update_rate> -->
+            <topic>${prefix}/joint_states</topic>
             <joint_name>${prefix}_B2C</joint_name>
             <joint_name>${prefix}_C2F</joint_name>
