Commit message: update controller and joint states plugins

File: PARAM/lbr_description/urdf/Grieel/LIMBERO.xacro (robot description, xacro)
@@ -11,8 +11,8 @@
   <!-- Use macro to define base and four limbs -->
   <xacro:base_macro/>
-  <xacro:limb_macro prefix="LF" parent="base_link" radius="45"/>
-  <xacro:limb_macro prefix="LH" parent="base_link" radius="135"/>
-  <xacro:limb_macro prefix="RH" parent="base_link" radius="225"/>
-  <xacro:limb_macro prefix="RF" parent="base_link" radius="315"/>
+  <xacro:limb_macro prefix="LF" parent="base_frame" radius="45"/>
+  <xacro:limb_macro prefix="LH" parent="base_frame" radius="135"/>
+  <xacro:limb_macro prefix="RH" parent="base_frame" radius="225"/>
+  <xacro:limb_macro prefix="RF" parent="base_frame" radius="315"/>
   <xacro:arg name="wheel_mode" default="true" />
   <!-- Grieel wheel mode -->
@@ -44,4 +44,5 @@
   <xacro:joint_state_macro prefix="RH"/>
   <xacro:joint_state_macro prefix="RF"/>
+  <xacro:include filename="$(find lbr_description)/urdf/Grieel/lbr_grieel_joint_state.xacro" />
   <xacro:joint_actuator_macro prefix="LF"/>
   <xacro:joint_actuator_macro prefix="LH"/>

File: PARAM/lbr_description/urdf/Grieel/grieel_gazebo_phisics.xacro (robot description, xacro)
@@ -20,6 +20,6 @@
         <xacro:unless value="$(arg wheel_mode)">
             <gazebo reference="${prefix}_gripper_Link">
-                <mu1>0.6</mu1>
-                <mu2>0.6</mu2>
+                <mu1>1.0</mu1>
+                <mu2>1.0</mu2>
                 <kp>1000000</kp>
                 <kd>1.0</kd>

File: PARAM/lbr_description/urdf/Grieel/lbr_base_description.xacro (robot description, xacro)
@@ -6,55 +6,61 @@
   name="LIMBERO_v1_8_Base" xmlns:xacro="http://ros.org/wiki/xacro">
   <xacro:macro name="base_macro">
-  <link
-    name="base_link">
-    <inertial>
-      <origin
-        xyz="0 0 -0.0030083"
-        rpy="0 0 0" />
-      <mass
-        value="3.1152" />
-      <inertia
-        ixx="0.0036482"
-        ixy="7.8081E-07"
-        ixz="1.7521E-06"
-        iyy="0.0062179"
-        iyz="-1.4424E-06"
-        izz="0.0034682" />
-    </inertial>
-    <visual>
-      <origin
-        xyz="0 0 0"
-        rpy="0 0 0" />
-      <geometry>
-        <mesh
-          filename="file://$(find lbr_description)/meshes/base.STL" scale="1.0 1.0 1.0"/>
-      </geometry>
-      <material
-        name="">
-        <color
-          rgba="0.2 0.2 0.2 1" />
-      </material>
-    </visual>
-    <collision>
-      <origin
-        xyz="0 0 0"
-        rpy="0 0 0" />
-      <geometry>
-        <mesh
-          filename="file://$(find lbr_description)/meshes/base.STL" scale="1.0 1.0 1.0"/>
-      </geometry>
-    </collision>
-  </link>
-  <gazebo reference="base_link">
-    <material>Gazebo/Black</material>
-    <visual>
-      <material>
-        <ambient>0.2 0.2 0.2 1</ambient>
-        <diffuse>0.2 0.2 0.2 1</diffuse>
-        <specular>0.01 0.01 0.01 1</specular>
-        <emissive>0.01 0.01 0.01 1</emissive>
-      </material>
-    </visual>
-  </gazebo>
+    <link
+      name="base_link">
+      <inertial>
+        <origin
+          xyz="0 0 -0.0030083"
+          rpy="0 0 0" />
+        <mass
+          value="3.1152" />
+        <inertia
+          ixx="0.0036482"
+          ixy="7.8081E-07"
+          ixz="1.7521E-06"
+          iyy="0.0062179"
+          iyz="-1.4424E-06"
+          izz="0.0034682" />
+      </inertial>
+      <visual>
+        <origin
+          xyz="0 0 0"
+          rpy="0 0 0" />
+        <geometry>
+          <mesh
+            filename="file://$(find lbr_description)/meshes/base.STL" scale="1.0 1.0 1.0"/>
+        </geometry>
+        <material
+          name="">
+          <color
+            rgba="0.2 0.2 0.2 1" />
+        </material>
+      </visual>
+      <collision>
+        <origin
+          xyz="0 0 0"
+          rpy="0 0 0" />
+        <geometry>
+          <mesh
+            filename="file://$(find lbr_description)/meshes/base.STL" scale="1.0 1.0 1.0"/>
+        </geometry>
+      </collision>
+    </link>
+    <gazebo reference="base_link">
+      <material>Gazebo/Black</material>
+      <visual>
+        <material>
+          <ambient>0.2 0.2 0.2 1</ambient>
+          <diffuse>0.2 0.2 0.2 1</diffuse>
+          <specular>0.01 0.01 0.01 1</specular>
+          <emissive>0.01 0.01 0.01 1</emissive>
+        </material>
+      </visual>
+    </gazebo>
+    <link name="base_frame"/>
+    <joint name="base_frame_joint" type="fixed">
+        <origin rpy="0 0 0" xyz="0 0 0"/>
+        <parent link="base_link" />
+        <child link="base_frame" />
+    </joint>
   </xacro:macro>
 </robot>

Commit message: 5th order polynomial + debug in wrist

File: PARAM/lbr_description/urdf/Grieel/LIMBERO.xacro (robot description, xacro)
@@ -7,12 +7,13 @@
   <xacro:include filename="$(find lbr_description)/urdf/Grieel/lbr_grieel_joint_actuation.xacro" />
   <xacro:include filename="$(find lbr_description)/urdf/Grieel/grieel_gazebo_phisics.xacro" />
+  <!-- <xacro:include filename="$(find lbr_description)/urdf/Grieel/lbr_grieel_plugins.xacro" /> -->
   <!-- <xacro:include filename="$(find lbr_description)/urdf/Grieel/lbr_grieel_transmission.xacro" /> -->
   <!-- <xacro:include filename="$(find lbr_description)/urdf/Grieel/lidar.xacro" /> -->
   <!-- Use macro to define base and four limbs -->
   <xacro:base_macro/>
-  <xacro:limb_macro prefix="LF" parent="base_frame" radius="45"/>
-  <xacro:limb_macro prefix="LH" parent="base_frame" radius="135"/>
-  <xacro:limb_macro prefix="RH" parent="base_frame" radius="225"/>
-  <xacro:limb_macro prefix="RF" parent="base_frame" radius="315"/>
+  <xacro:limb_macro prefix="LF" parent="base_link" radius="45"/>
+  <xacro:limb_macro prefix="LH" parent="base_link" radius="135"/>
+  <xacro:limb_macro prefix="RH" parent="base_link" radius="225"/>
+  <xacro:limb_macro prefix="RF" parent="base_link" radius="315"/>
   <xacro:arg name="wheel_mode" default="true" />
   <!-- Grieel wheel mode -->

File: PARAM/lbr_description/urdf/Grieel/lbr_base_description.xacro (robot description, xacro)
@@ -57,4 +57,5 @@
       </visual>
     </gazebo>
+<!--
     <link name="base_frame"/>
     <joint name="base_frame_joint" type="fixed">
@@ -62,5 +63,5 @@
         <parent link="base_link" />
         <child link="base_frame" />
-    </joint>
+    </joint> -->
   </xacro:macro>
 </robot>

File: PARAM/lbr_description/urdf/Grieel/lbr_grieel_joint_state.xacro (robot description, xacro)
@@ -14,5 +14,4 @@
             <!-- <update_rate>500</update_rate> -->
             <topic>/joint_states</topic>
-            <!-- <joint_name>world_base</joint_name> -->
             <joint_name>LF_B2C</joint_name>
             <joint_name>LF_C2F</joint_name>
