Commit message: implementing actuated fingers, controller missing
bullet engine is needed to use mimic joints

File: PARAM/lbr_description/urdf/Grieel/LIMBERO.xacro (robot description, xacro)
@@ -6,5 +6,5 @@
   <xacro:include filename="$(find lbr_description)/urdf/Grieel/grieel_joint_state.xacro" />
   <xacro:include filename="$(find lbr_description)/urdf/Grieel/lbr_grieel_joint_actuation.xacro" />
-  <xacro:include filename="$(find lbr_description)/urdf/Grieel/grieel_gazebo_phisics.xacro" />
+  <xacro:include filename="$(find lbr_description)/urdf/Grieel/grieel_gazebo_colors.xacro" />
   <!-- <xacro:include filename="$(find lbr_description)/urdf/Grieel/lbr_grieel_plugins.xacro" /> -->
   <!-- <xacro:include filename="$(find lbr_description)/urdf/Grieel/lbr_grieel_transmission.xacro" /> -->
@@ -54,7 +54,7 @@
   <xacro:transmission_macro prefix="RH"/>
   <xacro:transmission_macro prefix="RF"/> -->
-  <xacro:gazebo_phisics_macro prefix="LF"/>
-  <xacro:gazebo_phisics_macro prefix="LH"/>
-  <xacro:gazebo_phisics_macro prefix="RH"/>
-  <xacro:gazebo_phisics_macro prefix="RF"/>
+  <xacro:gazebo_colors_macro prefix="LF"/>
+  <xacro:gazebo_colors_macro prefix="LH"/>
+  <xacro:gazebo_colors_macro prefix="RH"/>
+  <xacro:gazebo_colors_macro prefix="RF"/>
 </robot>

File: PARAM/lbr_description/urdf/Grieel/grieel_finger_macro.xacro (robot description, xacro)
@@ -20,5 +20,5 @@
         <limit
         lower="0.0"
-        upper="${pi/3}"
+        upper="${pi/6}"
         effort="0.0"
         velocity="0.0" />
@@ -27,18 +27,18 @@
     <link
         name="${prefix}_${name}_phalanx1">
-        <!-- <inertial>
-        <origin
-            xyz="0.011821 8.7424E-07 4.3619E-14"
-            rpy="0 0 0" />
-        <mass
-            value="0.00824" />
-        <inertia
-            ixx="1.7943E-06"
-            ixy="-3.8552E-19"
-            ixz="7.4101E-19"
-            iyy="2.9379E-06"
-            iyz="-2.3646E-09"
-            izz="1.6633E-06" />
-        </inertial> -->
+        <inertial>
+            <origin
+                xyz="0.00162585 0.00031929 0.01672194"
+                rpy="0 0 0" />
+            <mass
+                value="0.003797793442763989" />
+            <inertia
+                ixx="3.31093803e-07"
+                ixy="3.15649096e-09"
+                ixz="-1.22740945e-09"
+                iyy="3.44910628e-07"
+                iyz="-4.29494199e-09"
+                izz="8.86398503e-08" />
+        </inertial>
         <visual>
         <origin
@@ -65,8 +65,23 @@
         </collision>
     </link>
+    <gazebo reference="${prefix}_${name}_phalanx1">
+        <material>Gazebo/Black</material>
+        <visual>
+            <material>
+                <ambient>0.2 0.2 0.2 1</ambient>
+                <diffuse>0.2 0.2 0.2 1</diffuse>
+                <specular>0.01 0.01 0.01 1</specular>
+                <emissive>0.01 0.01 0.01 1</emissive>
+            </material>
+        </visual>
+        <mu1>1.0</mu1>
+        <mu2>1.0</mu2>
+        <kp>1000000</kp>
+        <kd>1.0</kd>
+    </gazebo>
     <joint
         name="${prefix}_${name}_P12P2"
         type="revolute">
-        <mimic joint="${prefix}_F1_H2P1" multiplier="1" offset="0"/>
+        <mimic joint="${prefix}_F1_H2P1" multiplier="2" offset="0"/>
         <origin
         xyz="0 0 0.030654"
@@ -87,18 +102,18 @@
     <link
         name="${prefix}_${name}_phalanx2">
-        <!-- <inertial>
-        <origin
-            xyz="0.011821 8.7424E-07 4.3619E-14"
-            rpy="0 0 0" />
-        <mass
-            value="0.00824" />
-        <inertia
-            ixx="1.7943E-06"
-            ixy="-3.8552E-19"
-            ixz="7.4101E-19"
-            iyy="2.9379E-06"
-            iyz="-2.3646E-09"
-            izz="1.6633E-06" />
-        </inertial> -->
+        <inertial>
+            <origin
+                xyz="-0.00673704 0.00047222 0.01186178"
+                rpy="0 0 0" />
+            <mass
+                value="0.013082859723205855" />
+            <inertia
+                ixx="3.00003952e-06"
+                ixy="-6.39755832e-09"
+                ixz="-9.83815289e-08"
+                iyy="1.39153928e-06"
+                iyz="7.23067218e-09"
+                izz="2.30350901e-06" />
+        </inertial>
         <visual>
         <origin
@@ -125,8 +140,23 @@
         </collision>
     </link>
+    <gazebo reference="${prefix}_${name}_phalanx2">
+        <material>Gazebo/Black</material>
+        <visual>
+            <material>
+                <ambient>0.2 0.2 0.2 1</ambient>
+                <diffuse>0.2 0.2 0.2 1</diffuse>
+                <specular>0.01 0.01 0.01 1</specular>
+                <emissive>0.01 0.01 0.01 1</emissive>
+            </material>
+        </visual>
+        <mu1>1.0</mu1>
+        <mu2>1.0</mu2>
+        <kp>1000000</kp>
+        <kd>1.0</kd>
+    </gazebo>
    <joint
         name="${prefix}_${name}_P22P3"
         type="revolute">
-        <mimic joint="${prefix}_F1_H2P1" multiplier="1" offset="0"/>
+        <mimic joint="${prefix}_F1_H2P1" multiplier="3" offset="0"/>
         <origin
         xyz="0 0 0.028999"
@@ -147,18 +177,18 @@
     <link
         name="${prefix}_${name}_phalanx3">
-        <!-- <inertial>
-        <origin
-            xyz="0.011821 8.7424E-07 4.3619E-14"
-            rpy="0 0 0" />
-        <mass
-            value="0.00824" />
-        <inertia
-            ixx="1.7943E-06"
-            ixy="-3.8552E-19"
-            ixz="7.4101E-19"
-            iyy="2.9379E-06"
-            iyz="-2.3646E-09"
-            izz="1.6633E-06" />
-        </inertial> -->
+        <inertial>
+            <origin
+                xyz="-0.00232913 0.00061377 0.01268651"
+                rpy="0 0 0" />
+            <mass
+                value="0.0024217622661742476" />
+            <inertia
+                ixx="1.24811429e-07"
+                ixy="5.11516670e-10"
+                ixz="1.67264903e-08"
+                iyy="1.28312272e-07"
+                iyz="1.69572891e-09"
+                izz="4.48441736e-08" />
+        </inertial>
         <visual>
         <origin
@@ -185,4 +215,19 @@
         </collision>
     </link>
+    <gazebo reference="${prefix}_${name}_phalanx3">
+        <material>Gazebo/Black</material>
+        <visual>
+            <material>
+                <ambient>0.2 0.2 0.2 1</ambient>
+                <diffuse>0.2 0.2 0.2 1</diffuse>
+                <specular>0.01 0.01 0.01 1</specular>
+                <emissive>0.01 0.01 0.01 1</emissive>
+            </material>
+        </visual>
+        <mu1>1.0</mu1>
+        <mu2>1.0</mu2>
+        <kp>1000000</kp>
+        <kd>1.0</kd>
+    </gazebo>
   </xacro:macro>
 </robot>

File: PARAM/lbr_description/urdf/Grieel/grieel_first_finger_macro.xacro (robot description, xacro)
@@ -19,5 +19,5 @@
         <limit
         lower="0.0"
-        upper="${pi/3}"
+        upper="${pi/6}"
         effort="0.0"
         velocity="0.0" />
@@ -26,18 +26,18 @@
     <link
         name="${prefix}_${name}_phalanx1">
-        <!-- <inertial>
-        <origin
-            xyz="0.011821 8.7424E-07 4.3619E-14"
-            rpy="0 0 0" />
-        <mass
-            value="0.00824" />
-        <inertia
-            ixx="1.7943E-06"
-            ixy="-3.8552E-19"
-            ixz="7.4101E-19"
-            iyy="2.9379E-06"
-            iyz="-2.3646E-09"
-            izz="1.6633E-06" />
-        </inertial> -->
+        <inertial>
+            <origin
+                xyz="0.00162585 0.00031929 0.01672194"
+                rpy="0 0 0" />
+            <mass
+                value="0.003797793442763989" />
+            <inertia
+                ixx="3.31093803e-07"
+                ixy="3.15649096e-09"
+                ixz="-1.22740945e-09"
+                iyy="3.44910628e-07"
+                iyz="-4.29494199e-09"
+                izz="8.86398503e-08" />
+        </inertial>
         <visual>
         <origin
@@ -64,8 +64,23 @@
         </collision>
     </link>
+    <gazebo reference="${prefix}_${name}_phalanx1">
+        <material>Gazebo/Black</material>
+        <visual>
+            <material>
+                <ambient>0.2 0.2 0.2 1</ambient>
+                <diffuse>0.2 0.2 0.2 1</diffuse>
+                <specular>0.01 0.01 0.01 1</specular>
+                <emissive>0.01 0.01 0.01 1</emissive>
+            </material>
+        </visual>
+        <mu1>1.0</mu1>
+        <mu2>1.0</mu2>
+        <kp>1000000</kp>
+        <kd>1.0</kd>
+    </gazebo>
     <joint
         name="${prefix}_${name}_P12P2"
         type="revolute">
-        <mimic joint="${prefix}_F1_H2P1" multiplier="1" offset="0"/>
+        <mimic joint="${prefix}_F1_H2P1" multiplier="2" offset="0"/>
         <origin
         xyz="0 0 0.030654"
@@ -86,18 +101,18 @@
     <link
         name="${prefix}_${name}_phalanx2">
-        <!-- <inertial>
-        <origin
-            xyz="0.011821 8.7424E-07 4.3619E-14"
-            rpy="0 0 0" />
-        <mass
-            value="0.00824" />
-        <inertia
-            ixx="1.7943E-06"
-            ixy="-3.8552E-19"
-            ixz="7.4101E-19"
-            iyy="2.9379E-06"
-            iyz="-2.3646E-09"
-            izz="1.6633E-06" />
-        </inertial> -->
+        <inertial>
+            <origin
+                xyz="-0.00673704 0.00047222 0.01186178"
+                rpy="0 0 0" />
+            <mass
+                value="0.013082859723205855" />
+            <inertia
+                ixx="3.00003952e-06"
+                ixy="-6.39755832e-09"
+                ixz="-9.83815289e-08"
+                iyy="1.39153928e-06"
+                iyz="7.23067218e-09"
+                izz="2.30350901e-06" />
+        </inertial>
         <visual>
         <origin
@@ -124,8 +139,23 @@
         </collision>
     </link>
+    <gazebo reference="${prefix}_${name}_phalanx2">
+        <material>Gazebo/Black</material>
+        <visual>
+            <material>
+                <ambient>0.2 0.2 0.2 1</ambient>
+                <diffuse>0.2 0.2 0.2 1</diffuse>
+                <specular>0.01 0.01 0.01 1</specular>
+                <emissive>0.01 0.01 0.01 1</emissive>
+            </material>
+        </visual>
+        <mu1>1.0</mu1>
+        <mu2>1.0</mu2>
+        <kp>1000000</kp>
+        <kd>1.0</kd>
+    </gazebo>
    <joint
         name="${prefix}_${name}_P22P3"
         type="revolute">
-        <mimic joint="${prefix}_F1_H2P1" multiplier="1" offset="0"/>
+        <mimic joint="${prefix}_F1_H2P1" multiplier="3" offset="0"/>
         <origin
         xyz="0 0 0.028999"
@@ -146,18 +176,18 @@
     <link
         name="${prefix}_${name}_phalanx3">
-        <!-- <inertial>
-        <origin
-            xyz="0.011821 8.7424E-07 4.3619E-14"
-            rpy="0 0 0" />
-        <mass
-            value="0.00824" />
-        <inertia
-            ixx="1.7943E-06"
-            ixy="-3.8552E-19"
-            ixz="7.4101E-19"
-            iyy="2.9379E-06"
-            iyz="-2.3646E-09"
-            izz="1.6633E-06" />
-        </inertial> -->
+        <inertial>
+            <origin
+                xyz="-0.00232913 0.00061377 0.01268651"
+                rpy="0 0 0" />
+            <mass
+                value="0.0024217622661742476" />
+            <inertia
+                ixx="1.24811429e-07"
+                ixy="5.11516670e-10"
+                ixz="1.67264903e-08"
+                iyy="1.28312272e-07"
+                iyz="1.69572891e-09"
+                izz="4.48441736e-08" />
+        </inertial>
         <visual>
         <origin
@@ -184,4 +214,19 @@
         </collision>
     </link>
+    <gazebo reference="${prefix}_${name}_phalanx3">
+        <material>Gazebo/Black</material>
+        <visual>
+            <material>
+                <ambient>0.2 0.2 0.2 1</ambient>
+                <diffuse>0.2 0.2 0.2 1</diffuse>
+                <specular>0.01 0.01 0.01 1</specular>
+                <emissive>0.01 0.01 0.01 1</emissive>
+            </material>
+        </visual>
+        <mu1>1.0</mu1>
+        <mu2>1.0</mu2>
+        <kp>1000000</kp>
+        <kd>1.0</kd>
+    </gazebo>
   </xacro:macro>
 </robot>

File: PARAM/lbr_description/urdf/Grieel/grieel_gripper_splitted.xacro (robot description, xacro)
@@ -27,18 +27,18 @@
     <link
         name="${prefix}_hand_Link">
-        <!-- <inertial>
+        <inertial>
         <origin
-            xyz="0.011821 8.7424E-07 4.3619E-14"
+            xyz="0.05982052 -0.00756175 0.00448521"
             rpy="0 0 0" />
         <mass
-            value="0.00824" />
+            value="0.125" />
         <inertia
-            ixx="1.7943E-06"
-            ixy="-3.8552E-19"
-            ixz="7.4101E-19"
-            iyy="2.9379E-06"
-            iyz="-2.3646E-09"
-            izz="1.6633E-06" />
-        </inertial> -->
+            ixx="1.00731433e-04"
+            ixy="-1.43025925e-05"
+            ixz="5.35158888e-06"
+            iyy="8.56906244e-05"
+            iyz="-2.56859397e-06"
+            izz="1.13275414e-04" />
+        </inertial>
         <visual>
         <origin

File: PARAM/lbr_description/urdf/Grieel/lbr_grieel_joint_state.xacro (robot description, xacro)
@@ -21,4 +21,28 @@
             <joint_name>LF_wristV</joint_name>
             <joint_name>LF_driving</joint_name>
+            <joint_name>LF_F1_H2P1</joint_name>
+            <joint_name>LF_F1_P12P2</joint_name>
+            <joint_name>LF_F1_P22P3</joint_name>
+            <joint_name>LF_F2_H2P1</joint_name>
+            <joint_name>LF_F2_P12P2</joint_name>
+            <joint_name>LF_F2_P22P3</joint_name>
+            <joint_name>LF_F3_H2P1</joint_name>
+            <joint_name>LF_F3_P12P2</joint_name>
+            <joint_name>LF_F3_P22P3</joint_name>
+            <joint_name>LF_F4_H2P1</joint_name>
+            <joint_name>LF_F4_P12P2</joint_name>
+            <joint_name>LF_F4_P22P3</joint_name>
+            <joint_name>LF_F5_H2P1</joint_name>
+            <joint_name>LF_F5_P12P2</joint_name>
+            <joint_name>LF_F5_P22P3</joint_name>
+            <joint_name>LF_F6_H2P1</joint_name>
+            <joint_name>LF_F6_P12P2</joint_name>
+            <joint_name>LF_F6_P22P3</joint_name>
+            <joint_name>LF_F7_H2P1</joint_name>
+            <joint_name>LF_F7_P12P2</joint_name>
+            <joint_name>LF_F7_P22P3</joint_name>
+            <joint_name>LF_F8_H2P1</joint_name>
+            <joint_name>LF_F8_P12P2</joint_name>
+            <joint_name>LF_F8_P22P3</joint_name>
             <joint_name>LH_B2C</joint_name>
             <joint_name>LH_C2F</joint_name>
@@ -28,4 +52,28 @@
             <joint_name>LH_wristV</joint_name>
             <joint_name>LH_driving</joint_name>
+            <joint_name>LH_F1_H2P1</joint_name>
+            <joint_name>LH_F1_P12P2</joint_name>
+            <joint_name>LH_F1_P22P3</joint_name>
+            <joint_name>LH_F2_H2P1</joint_name>
+            <joint_name>LH_F2_P12P2</joint_name>
+            <joint_name>LH_F2_P22P3</joint_name>
+            <joint_name>LH_F3_H2P1</joint_name>
+            <joint_name>LH_F3_P12P2</joint_name>
+            <joint_name>LH_F3_P22P3</joint_name>
+            <joint_name>LH_F4_H2P1</joint_name>
+            <joint_name>LH_F4_P12P2</joint_name>
+            <joint_name>LH_F4_P22P3</joint_name>
+            <joint_name>LH_F5_H2P1</joint_name>
+            <joint_name>LH_F5_P12P2</joint_name>
+            <joint_name>LH_F5_P22P3</joint_name>
+            <joint_name>LH_F6_H2P1</joint_name>
+            <joint_name>LH_F6_P12P2</joint_name>
+            <joint_name>LH_F6_P22P3</joint_name>
+            <joint_name>LH_F7_H2P1</joint_name>
+            <joint_name>LH_F7_P12P2</joint_name>
+            <joint_name>LH_F7_P22P3</joint_name>
+            <joint_name>LH_F8_H2P1</joint_name>
+            <joint_name>LH_F8_P12P2</joint_name>
+            <joint_name>LH_F8_P22P3</joint_name>
             <joint_name>RH_B2C</joint_name>
             <joint_name>RH_C2F</joint_name>
@@ -35,4 +83,28 @@
             <joint_name>RH_wristV</joint_name>
             <joint_name>RH_driving</joint_name>
+            <joint_name>RH_F1_H2P1</joint_name>
+            <joint_name>RH_F1_P12P2</joint_name>
+            <joint_name>RH_F1_P22P3</joint_name>
+            <joint_name>RH_F2_H2P1</joint_name>
+            <joint_name>RH_F2_P12P2</joint_name>
+            <joint_name>RH_F2_P22P3</joint_name>
+            <joint_name>RH_F3_H2P1</joint_name>
+            <joint_name>RH_F3_P12P2</joint_name>
+            <joint_name>RH_F3_P22P3</joint_name>
+            <joint_name>RH_F4_H2P1</joint_name>
+            <joint_name>RH_F4_P12P2</joint_name>
+            <joint_name>RH_F4_P22P3</joint_name>
+            <joint_name>RH_F5_H2P1</joint_name>
+            <joint_name>RH_F5_P12P2</joint_name>
+            <joint_name>RH_F5_P22P3</joint_name>
+            <joint_name>RH_F6_H2P1</joint_name>
+            <joint_name>RH_F6_P12P2</joint_name>
+            <joint_name>RH_F6_P22P3</joint_name>
+            <joint_name>RH_F7_H2P1</joint_name>
+            <joint_name>RH_F7_P12P2</joint_name>
+            <joint_name>RH_F7_P22P3</joint_name>
+            <joint_name>RH_F8_H2P1</joint_name>
+            <joint_name>RH_F8_P12P2</joint_name>
+            <joint_name>RH_F8_P22P3</joint_name>
             <joint_name>RF_B2C</joint_name>
             <joint_name>RF_C2F</joint_name>
@@ -42,4 +114,28 @@
             <joint_name>RF_wristV</joint_name>
             <joint_name>RF_driving</joint_name>
+            <joint_name>RF_F1_H2P1</joint_name>
+            <joint_name>RF_F1_P12P2</joint_name>
+            <joint_name>RF_F1_P22P3</joint_name>
+            <joint_name>RF_F2_H2P1</joint_name>
+            <joint_name>RF_F2_P12P2</joint_name>
+            <joint_name>RF_F2_P22P3</joint_name>
+            <joint_name>RF_F3_H2P1</joint_name>
+            <joint_name>RF_F3_P12P2</joint_name>
+            <joint_name>RF_F3_P22P3</joint_name>
+            <joint_name>RF_F4_H2P1</joint_name>
+            <joint_name>RF_F4_P12P2</joint_name>
+            <joint_name>RF_F4_P22P3</joint_name>
+            <joint_name>RF_F5_H2P1</joint_name>
+            <joint_name>RF_F5_P12P2</joint_name>
+            <joint_name>RF_F5_P22P3</joint_name>
+            <joint_name>RF_F6_H2P1</joint_name>
+            <joint_name>RF_F6_P12P2</joint_name>
+            <joint_name>RF_F6_P22P3</joint_name>
+            <joint_name>RF_F7_H2P1</joint_name>
+            <joint_name>RF_F7_P12P2</joint_name>
+            <joint_name>RF_F7_P22P3</joint_name>
+            <joint_name>RF_F8_H2P1</joint_name>
+            <joint_name>RF_F8_P12P2</joint_name>
+            <joint_name>RF_F8_P22P3</joint_name>
         </plugin>
     </gazebo>
