Commit message: implement GRIEEL open/close ros2_control

File: PARAM/lbr_description/urdf/Grieel/LIMBERO.xacro (robot description, xacro)
@@ -2,4 +2,5 @@
   <xacro:include filename="$(find lbr_description)/urdf/Grieel/lbr_base_description.xacro" />
   <xacro:include filename="$(find lbr_description)/urdf/Grieel/lbr_limb_description.xacro" />
+  <xacro:include filename="$(find lbr_description)/urdf/Grieel/grieel_gazebo_ros2_control.xacro" />
   <!-- <xacro:include filename="$(find lbr_description)/urdf/Grieel/lbr_gazebo.xacro" /> -->
   <!-- <xacro:include filename="$(find lbr_description)/urdf/Grieel/lbr_ros2_control.xacro" /> -->
@@ -59,9 +60,5 @@
   <xacro:gazebo_colors_macro prefix="RH"/>
   <xacro:gazebo_colors_macro prefix="RF"/>
-  <gazebo>
-      <plugin name="gz_ros2_control::GazeboSimROS2ControlPlugin" filename="libgz_ros2_control-system.so">
-            <parameters>$(find lbr_description)/config/grieel_controller.yaml</parameters>
-      </plugin>
-  </gazebo>
+  <xacro:load_gazebo_sim_ros2_control_plugin/>
   <xacro:grieel_ros2_control_macro prefix="LF"/>
   <xacro:grieel_ros2_control_macro prefix="LH"/>

File: PARAM/lbr_description/urdf/Grieel/grieel_finger_macro.xacro (robot description, xacro)
@@ -21,7 +21,7 @@
         lower="0.0"
         upper="${pi/6}"
-        effort="10.0"
+        effort="50.0"
         velocity="10.0" />
-        <dynamics damping="0.1" friction="0.3"/>
+        <dynamics damping="0.05" friction="0.1"/>
     </joint>
     <link
@@ -96,7 +96,7 @@
         lower="${-pi/3}"
         upper="${pi*3/2}"
-        effort="10.0"
+        effort="50.0"
         velocity="10.0" />
-        <dynamics damping="0.1" friction="0.3"/>
+        <dynamics damping="0.05" friction="0.1"/>
     </joint>
     <link
@@ -171,7 +171,7 @@
         lower="${-pi/3}"
         upper="${pi*3/2}"
-        effort="10.0"
+        effort="50.0"
         velocity="10.0" />
-        <dynamics damping="0.1" friction="0.3"/>
+        <dynamics damping="0.05" friction="0.1"/>
     </joint>
     <link

File: PARAM/lbr_description/urdf/Grieel/grieel_first_finger_macro.xacro (robot description, xacro)
@@ -20,7 +20,7 @@
         lower="0.0"
         upper="${pi/6}"
-        effort="10.0"
+        effort="50.0"
         velocity="10.0" />
-        <dynamics damping="0.1" friction="0.3"/>
+        <dynamics damping="0.05" friction="0.1"/>
     </joint>
     <link
@@ -95,7 +95,7 @@
         lower="${-pi/3}"
         upper="${pi*3/2}"
-        effort="10.0"
+        effort="50.0"
         velocity="10.0" />
-        <dynamics damping="0.1" friction="0.3"/>
+        <dynamics damping="0.05" friction="0.1"/>
     </joint>
     <link
@@ -170,7 +170,7 @@
         lower="${-pi/3}"
         upper="${pi*3/2}"
-        effort="10.0"
+        effort="50.0"
         velocity="10.0" />
-        <dynamics damping="0.1" friction="0.3"/>
+        <dynamics damping="0.05" friction="0.1"/>
     </joint>
     <link

File: PARAM/lbr_description/urdf/Grieel/grieel_ros2_control.xacro (robot description, xacro)
@@ -7,99 +7,148 @@
       </hardware>
       <joint name="${prefix}_F1_H2P1">
-        <command_interface name="position"/>
+        <command_interface name="position">
+                    <param name="min">0.0</param>
+                    <param name="max">0.52359877559829887308</param>
+        </command_interface>
         <state_interface name="position"/>
         <state_interface name="velocity"/>
       </joint>
       <joint name="${prefix}_F1_P12P2">
-        <state_interface name="position"/>
-        <state_interface name="velocity"/>
+          <param name="mimic">${prefix}_F1_H2P1</param>
+          <param name="multiplier">2.0</param>
+          <state_interface name="position"/>
+          <state_interface name="velocity"/>
       </joint>
       <joint name="${prefix}_F1_P22P3">
-        <state_interface name="position"/>
-        <state_interface name="velocity"/>
+          <param name="mimic">${prefix}_F1_H2P1</param>
+          <param name="multiplier">3.0</param>
+          <state_interface name="position"/>
+          <state_interface name="velocity"/>
       </joint>
       <joint name="${prefix}_F2_H2P1">
-        <state_interface name="position"/>
-        <state_interface name="velocity"/>
+          <param name="mimic">${prefix}_F1_H2P1</param>
+          <param name="multiplier">1.0</param>
+          <state_interface name="position"/>
+          <state_interface name="velocity"/>
       </joint>
       <joint name="${prefix}_F2_P12P2">
-        <state_interface name="position"/>
-        <state_interface name="velocity"/>
+          <param name="mimic">${prefix}_F1_H2P1</param>
+          <param name="multiplier">2.0</param>
+          <state_interface name="position"/>
+          <state_interface name="velocity"/>
       </joint>
       <joint name="${prefix}_F2_P22P3">
-        <state_interface name="position"/>
-        <state_interface name="velocity"/>
+          <param name="mimic">${prefix}_F1_H2P1</param>
+          <param name="multiplier">3.0</param>
+          <state_interface name="position"/>
+          <state_interface name="velocity"/>
       </joint>
       <joint name="${prefix}_F3_H2P1">
-        <state_interface name="position"/>
-        <state_interface name="velocity"/>
+          <param name="mimic">${prefix}_F1_H2P1</param>
+          <param name="multiplier">1.0</param>
+          <state_interface name="position"/>
+          <state_interface name="velocity"/>
       </joint>
       <joint name="${prefix}_F3_P12P2">
-        <state_interface name="position"/>
-        <state_interface name="velocity"/>
+          <param name="mimic">${prefix}_F1_H2P1</param>
+          <param name="multiplier">2.0</param>
+          <state_interface name="position"/>
+          <state_interface name="velocity"/>
       </joint>
       <joint name="${prefix}_F3_P22P3">
-        <state_interface name="position"/>
-        <state_interface name="velocity"/>
+          <param name="mimic">${prefix}_F1_H2P1</param>
+          <param name="multiplier">3.0</param>
+          <state_interface name="position"/>
+          <state_interface name="velocity"/>
       </joint>
       <joint name="${prefix}_F4_H2P1">
-        <state_interface name="position"/>
-        <state_interface name="velocity"/>
+          <param name="mimic">${prefix}_F1_H2P1</param>
+          <param name="multiplier">1.0</param>
+          <state_interface name="position"/>
+          <state_interface name="velocity"/>
       </joint>
       <joint name="${prefix}_F4_P12P2">
-        <state_interface name="position"/>
-        <state_interface name="velocity"/>
+          <param name="mimic">${prefix}_F1_H2P1</param>
+          <param name="multiplier">2.0</param>
+          <state_interface name="position"/>
+          <state_interface name="velocity"/>
       </joint>
       <joint name="${prefix}_F4_P22P3">
-        <state_interface name="position"/>
-        <state_interface name="velocity"/>
+          <param name="mimic">${prefix}_F1_H2P1</param>
+          <param name="multiplier">3.0</param>
+          <state_interface name="position"/>
+          <state_interface name="velocity"/>
       </joint>
       <joint name="${prefix}_F5_H2P1">
-        <state_interface name="position"/>
-        <state_interface name="velocity"/>
+          <param name="mimic">${prefix}_F1_H2P1</param>
+          <param name="multiplier">1.0</param>
+          <state_interface name="position"/>
+          <state_interface name="velocity"/>
       </joint>
       <joint name="${prefix}_F5_P12P2">
-        <state_interface name="position"/>
-        <state_interface name="velocity"/>
+          <param name="mimic">${prefix}_F1_H2P1</param>
+          <param name="multiplier">2.0</param>
+          <state_interface name="position"/>
+          <state_interface name="velocity"/>
       </joint>
       <joint name="${prefix}_F5_P22P3">
-        <state_interface name="position"/>
-        <state_interface name="velocity"/>
+          <param name="mimic">${prefix}_F1_H2P1</param>
+          <param name="multiplier">3.0</param>
+          <state_interface name="position"/>
+          <state_interface name="velocity"/>
       </joint>
       <joint name="${prefix}_F6_H2P1">
-        <state_interface name="position"/>
-        <state_interface name="velocity"/>
+          <param name="mimic">${prefix}_F1_H2P1</param>
+          <param name="multiplier">1.0</param>
+          <state_interface name="position"/>
+          <state_interface name="velocity"/>
       </joint>
       <joint name="${prefix}_F6_P12P2">
-        <state_interface name="position"/>
-        <state_interface name="velocity"/>
+          <param name="mimic">${prefix}_F1_H2P1</param>
+          <param name="multiplier">2.0</param>
+          <state_interface name="position"/>
+          <state_interface name="velocity"/>
       </joint>
       <joint name="${prefix}_F6_P22P3">
-        <state_interface name="position"/>
-        <state_interface name="velocity"/>
+          <param name="mimic">${prefix}_F1_H2P1</param>
+          <param name="multiplier">3.0</param>
+          <state_interface name="position"/>
+          <state_interface name="velocity"/>
       </joint>
       <joint name="${prefix}_F7_H2P1">
-        <state_interface name="position"/>
-        <state_interface name="velocity"/>
+          <param name="mimic">${prefix}_F1_H2P1</param>
+          <param name="multiplier">1.0</param>
+          <state_interface name="position"/>
+          <state_interface name="velocity"/>
       </joint>
       <joint name="${prefix}_F7_P12P2">
-        <state_interface name="position"/>
-        <state_interface name="velocity"/>
+          <param name="mimic">${prefix}_F1_H2P1</param>
+          <param name="multiplier">2.0</param>
+          <state_interface name="position"/>
+          <state_interface name="velocity"/>
       </joint>
       <joint name="${prefix}_F7_P22P3">
-        <state_interface name="position"/>
-        <state_interface name="velocity"/>
+          <param name="mimic">${prefix}_F1_H2P1</param>
+          <param name="multiplier">3.0</param>
+          <state_interface name="position"/>
+          <state_interface name="velocity"/>
       </joint>
       <joint name="${prefix}_F8_H2P1">
-        <state_interface name="position"/>
-        <state_interface name="velocity"/>
+          <param name="mimic">${prefix}_F1_H2P1</param>
+          <param name="multiplier">1.0</param>
+          <state_interface name="position"/>
+          <state_interface name="velocity"/>
       </joint>
       <joint name="${prefix}_F8_P12P2">
-        <state_interface name="position"/>
-        <state_interface name="velocity"/>
+          <param name="mimic">${prefix}_F1_H2P1</param>
+          <param name="multiplier">2.0</param>
+          <state_interface name="position"/>
+          <state_interface name="velocity"/>
       </joint>
       <joint name="${prefix}_F8_P22P3">
-        <state_interface name="position"/>
-        <state_interface name="velocity"/>
+          <param name="mimic">${prefix}_F1_H2P1</param>
+          <param name="multiplier">3.0</param>
+          <state_interface name="position"/>
+          <state_interface name="velocity"/>
       </joint>
     </ros2_control>

File: PARAM/lbr_description/urdf/Grieel/lbr_grieel_joint_state.xacro (robot description, xacro)
@@ -21,5 +21,5 @@
             <joint_name>LF_wristV</joint_name>
             <joint_name>LF_driving</joint_name>
-            <joint_name>LF_F1_H2P1</joint_name>
+            <!-- <joint_name>LF_F1_H2P1</joint_name>
             <joint_name>LF_F1_P12P2</joint_name>
             <joint_name>LF_F1_P22P3</joint_name>
@@ -44,5 +44,5 @@
             <joint_name>LF_F8_H2P1</joint_name>
             <joint_name>LF_F8_P12P2</joint_name>
-            <joint_name>LF_F8_P22P3</joint_name>
+            <joint_name>LF_F8_P22P3</joint_name> -->
             <joint_name>LH_B2C</joint_name>
             <joint_name>LH_C2F</joint_name>
@@ -52,5 +52,5 @@
             <joint_name>LH_wristV</joint_name>
             <joint_name>LH_driving</joint_name>
-            <joint_name>LH_F1_H2P1</joint_name>
+            <!-- <joint_name>LH_F1_H2P1</joint_name>
             <joint_name>LH_F1_P12P2</joint_name>
             <joint_name>LH_F1_P22P3</joint_name>
@@ -75,5 +75,5 @@
             <joint_name>LH_F8_H2P1</joint_name>
             <joint_name>LH_F8_P12P2</joint_name>
-            <joint_name>LH_F8_P22P3</joint_name>
+            <joint_name>LH_F8_P22P3</joint_name> -->
             <joint_name>RH_B2C</joint_name>
             <joint_name>RH_C2F</joint_name>
@@ -83,5 +83,5 @@
             <joint_name>RH_wristV</joint_name>
             <joint_name>RH_driving</joint_name>
-            <joint_name>RH_F1_H2P1</joint_name>
+            <!-- <joint_name>RH_F1_H2P1</joint_name>
             <joint_name>RH_F1_P12P2</joint_name>
             <joint_name>RH_F1_P22P3</joint_name>
@@ -106,5 +106,5 @@
             <joint_name>RH_F8_H2P1</joint_name>
             <joint_name>RH_F8_P12P2</joint_name>
-            <joint_name>RH_F8_P22P3</joint_name>
+            <joint_name>RH_F8_P22P3</joint_name> -->
             <joint_name>RF_B2C</joint_name>
             <joint_name>RF_C2F</joint_name>
@@ -114,5 +114,5 @@
             <joint_name>RF_wristV</joint_name>
             <joint_name>RF_driving</joint_name>
-            <joint_name>RF_F1_H2P1</joint_name>
+            <!-- <joint_name>RF_F1_H2P1</joint_name>
             <joint_name>RF_F1_P12P2</joint_name>
             <joint_name>RF_F1_P22P3</joint_name>
@@ -137,5 +137,5 @@
             <joint_name>RF_F8_H2P1</joint_name>
             <joint_name>RF_F8_P12P2</joint_name>
-            <joint_name>RF_F8_P22P3</joint_name>
+            <joint_name>RF_F8_P22P3</joint_name> -->
         </plugin>
     </gazebo>

Commit message: updates and debug

File: PARAM/lbr_description/urdf/Grieel/LIMBERO.xacro (robot description, xacro)
@@ -47,5 +47,5 @@
   <xacro:joint_state_macro prefix="RH"/>
   <xacro:joint_state_macro prefix="RF"/>
-  <xacro:include filename="$(find lbr_description)/urdf/Grieel/lbr_grieel_joint_state.xacro" />
+  <!-- <xacro:include filename="$(find lbr_description)/urdf/Grieel/lbr_grieel_joint_state.xacro" /> -->
   <xacro:joint_actuator_macro prefix="LF"/>
   <xacro:joint_actuator_macro prefix="LH"/>

File: PARAM/lbr_description/urdf/Grieel/grieel_gripper_description.xacro (robot description, xacro)
@@ -7,4 +7,6 @@
   <xacro:macro name="grieel_gripper_macro" params="prefix parent">
   <xacro:include filename="$(find lbr_description)/urdf/Grieel/grieel_gripper_splitted.xacro" />
+    <xacro:property name="friction" value="0.1"/>
+    <xacro:property name="damping" value="0.05"/>
     <joint
       name="${prefix}_E2grieel"
@@ -122,5 +124,5 @@
       effort="8.0"
       velocity="4.0" />
-    <dynamics damping="0.1" friction="0.4"/>
+    <dynamics damping="${damping}" friction="${friction}"/>
   </joint>
   <link
@@ -181,5 +183,5 @@
       effort="8.0"
       velocity="4.0" />
-    <dynamics damping="0.1" friction="0.4"/>
+    <dynamics damping="${damping}" friction="${friction}"/>
   </joint>
   <!-- <link

File: PARAM/lbr_description/urdf/Grieel/grieel_joint_state.xacro (robot description, xacro)
@@ -13,18 +13,17 @@
         <gazebo>
             <plugin name="gz::sim::systems::JointStatePublisher" filename="gz-sim-joint-state-publisher-system">
-            <!-- <ros>
-                <namespace>${prefix}</namespace>
-                <remapping>~/out:=joint_states</remapping>
-            </ros> -->
-            <!-- <update_rate>500</update_rate> -->
-            <topic>${prefix}/joint_states</topic>
-            <joint_name>${prefix}_B2C</joint_name>
-            <joint_name>${prefix}_C2F</joint_name>
-            <joint_name>${prefix}_F2T</joint_name>
-            <joint_name>${prefix}_T2E</joint_name>
-            <joint_name>${prefix}_wristH</joint_name>
-            <joint_name>${prefix}_wristV</joint_name>
-            <joint_name>${prefix}_driving</joint_name>
-            <!-- <joint_name>${prefix}_F1_H2P1</joint_name> -->
+                <!-- <ros>
+                    <namespace>${prefix}</namespace>
+                    <remapping>~/out:=joint_states</remapping>
+                </ros> -->
+                <topic>${prefix}/joint_states</topic>
+                <joint_name>${prefix}_B2C</joint_name>
+                <joint_name>${prefix}_C2F</joint_name>
+                <joint_name>${prefix}_F2T</joint_name>
+                <joint_name>${prefix}_T2E</joint_name>
+                <joint_name>${prefix}_wristH</joint_name>
+                <joint_name>${prefix}_wristV</joint_name>
+                <joint_name>${prefix}_driving</joint_name>
+                <!-- <joint_name>${prefix}_F1_H2P1</joint_name> -->
             </plugin>
         </gazebo>

File: PARAM/lbr_description/urdf/Grieel/lbr_limb_description.xacro (robot description, xacro)
@@ -6,4 +6,6 @@
   name="LIMBERO_v1_7_Limb" xmlns:xacro="http://ros.org/wiki/xacro">
   <xacro:macro name="limb_macro" params="prefix parent radius">
+    <xacro:property name="friction" value="0.1"/>
+    <xacro:property name="damping" value="0.05"/>
     <joint
       name="${prefix}_joint"
@@ -114,5 +116,5 @@
         effort="16.0"
         velocity="3.0" />
-      <dynamics damping="0.1" friction="0.4"/>
+      <dynamics damping="${damping}" friction="${friction}"/>
     </joint>
     <!-- <transmission name="${prefix}_B2C_transmission">
@@ -183,5 +185,5 @@
         effort="16.0"
         velocity="5.0" />
-      <dynamics damping="0.1" friction="0.4"/>
+      <dynamics damping="${damping}" friction="${friction}"/>
     </joint>
     <!-- <transmission name="${prefix}_C2F_transmission">
@@ -252,5 +254,5 @@
         effort="10.0"
         velocity="5.0" />
-      <dynamics damping="0.1" friction="0.4"/>
+      <dynamics damping="${damping}" friction="${friction}"/>
       <initial_position value="${pi/2}"/>
     </joint>
@@ -322,5 +324,5 @@
         effort="8.0"
         velocity="4.0" />
-      <dynamics damping="0.1" friction="0.4"/>
+      <dynamics damping="${damping}" friction="${friction}"/>
     </joint>
     <!-- <transmission name="${prefix}_T2E_transmission">
