Commit message: wip finger implementation

File: PARAM/lbr_description/urdf/Grieel/grieel_finger_macro.xacro (robot description, xacro)
@@ -21,7 +21,7 @@
         lower="0.0"
         upper="${pi/6}"
-        effort="0.0"
-        velocity="0.0" />
-        <dynamics damping="0.1" friction="0.4"/>
+        effort="10.0"
+        velocity="10.0" />
+        <dynamics damping="0.1" friction="0.3"/>
     </joint>
     <link
@@ -96,7 +96,7 @@
         lower="${-pi/3}"
         upper="${pi*3/2}"
-        effort="0.0"
-        velocity="0.0" />
-        <dynamics damping="0.1" friction="0.4"/>
+        effort="10.0"
+        velocity="10.0" />
+        <dynamics damping="0.1" friction="0.3"/>
     </joint>
     <link
@@ -171,7 +171,7 @@
         lower="${-pi/3}"
         upper="${pi*3/2}"
-        effort="0.0"
-        velocity="0.0" />
-        <dynamics damping="0.1" friction="0.4"/>
+        effort="10.0"
+        velocity="10.0" />
+        <dynamics damping="0.1" friction="0.3"/>
     </joint>
     <link

File: PARAM/lbr_description/urdf/Grieel/grieel_first_finger_macro.xacro (robot description, xacro)
@@ -20,7 +20,7 @@
         lower="0.0"
         upper="${pi/6}"
-        effort="0.0"
-        velocity="0.0" />
-        <dynamics damping="0.1" friction="0.4"/>
+        effort="10.0"
+        velocity="10.0" />
+        <dynamics damping="0.1" friction="0.3"/>
     </joint>
     <link
@@ -95,7 +95,7 @@
         lower="${-pi/3}"
         upper="${pi*3/2}"
-        effort="0.0"
-        velocity="0.0" />
-        <dynamics damping="0.1" friction="0.4"/>
+        effort="10.0"
+        velocity="10.0" />
+        <dynamics damping="0.1" friction="0.3"/>
     </joint>
     <link
@@ -170,7 +170,7 @@
         lower="${-pi/3}"
         upper="${pi*3/2}"
-        effort="0.0"
-        velocity="0.0" />
-        <dynamics damping="0.1" friction="0.4"/>
+        effort="10.0"
+        velocity="10.0" />
+        <dynamics damping="0.1" friction="0.3"/>
     </joint>
     <link

File: PARAM/lbr_description/urdf/Grieel/grieel_joint_state.xacro (robot description, xacro)
@@ -26,4 +26,5 @@
             <joint_name>${prefix}_wristV</joint_name>
             <joint_name>${prefix}_driving</joint_name>
+            <joint_name>${prefix}_F1_H2P1</joint_name>
             </plugin>
         </gazebo>

File: PARAM/lbr_description/urdf/Grieel/lbr_grieel_joint_actuation.xacro (robot description, xacro)
@@ -52,4 +52,9 @@
                 <joint_name>${prefix}_driving</joint_name>
             </plugin>
+            <plugin filename="gz-sim-apply-joint-force-system"
+                        name="gz::sim::systems::ApplyJointForce">
+                <topic>{prefix}_F1_H2P1/joint_torque</topic>
+                <joint_name>${prefix}_F1_H2P1</joint_name>
+            </plugin>
         </gazebo>
     </xacro:macro>

File: PARAM/lbr_description/urdf/Grieel/lbr_limb_description.xacro (robot description, xacro)
@@ -253,4 +253,5 @@
         velocity="5.0" />
       <dynamics damping="0.1" friction="0.4"/>
+      <initial_position value="${pi/2}"/>
     </joint>
     <!-- <transmission name="${prefix}_F2T_transmission">

Commit message: ros2_control implementation

File: PARAM/lbr_description/urdf/Grieel/grieel_finger_macro.xacro (robot description, xacro)
@@ -6,4 +6,8 @@
   name="assembled_gripper_mode" xmlns:xacro="http://ros.org/wiki/xacro">
   <xacro:arg name="not_first_finger" default="false" />
+  <xacro:property name="ambient" value="0.2 0.2 0.2 1"/>
+  <xacro:property name="diffuse" value="0.2 0.2 0.2 1"/>
+  <xacro:property name="specular" value="0.01 0.01 0.01 1"/>
+  <xacro:property name="emissive" value="0.01 0.01 0.01 1"/>
   <xacro:macro name="grieel_gripper_finger_macro" params="prefix name *origin">
     <joint
@@ -69,8 +73,8 @@
         <visual>
             <material>
-                <ambient>0.2 0.2 0.2 1</ambient>
-                <diffuse>0.2 0.2 0.2 1</diffuse>
-                <specular>0.01 0.01 0.01 1</specular>
-                <emissive>0.01 0.01 0.01 1</emissive>
+                <ambient>${ambient}</ambient>
+                <diffuse>${diffuse}</diffuse>
+                <specular>${specular}</specular>
+                <emissive>${emissive}</emissive>
             </material>
         </visual>
@@ -144,8 +148,8 @@
         <visual>
             <material>
-                <ambient>0.2 0.2 0.2 1</ambient>
-                <diffuse>0.2 0.2 0.2 1</diffuse>
-                <specular>0.01 0.01 0.01 1</specular>
-                <emissive>0.01 0.01 0.01 1</emissive>
+                <ambient>${ambient}</ambient>
+                <diffuse>${diffuse}</diffuse>
+                <specular>${specular}</specular>
+                <emissive>${emissive}</emissive>
             </material>
         </visual>
@@ -219,8 +223,8 @@
         <visual>
             <material>
-                <ambient>0.2 0.2 0.2 1</ambient>
-                <diffuse>0.2 0.2 0.2 1</diffuse>
-                <specular>0.01 0.01 0.01 1</specular>
-                <emissive>0.01 0.01 0.01 1</emissive>
+                <ambient>${ambient}</ambient>
+                <diffuse>${diffuse}</diffuse>
+                <specular>${specular}</specular>
+                <emissive>${emissive}</emissive>
             </material>
         </visual>

File: PARAM/lbr_description/urdf/Grieel/grieel_first_finger_macro.xacro (robot description, xacro)
@@ -5,5 +5,8 @@
 <robot
   name="assembled_gripper_mode" xmlns:xacro="http://ros.org/wiki/xacro">
-  <xacro:arg name="not_first_finger" default="false" />
+  <xacro:property name="ambient" value="0.2 0.2 0.2 1"/>
+  <xacro:property name="diffuse" value="0.2 0.2 0.2 1"/>
+  <xacro:property name="specular" value="0.01 0.01 0.01 1"/>
+  <xacro:property name="emissive" value="0.01 0.01 0.01 1"/>
   <xacro:macro name="grieel_gripper_first_finger_macro" params="prefix name *origin">
     <joint
@@ -68,8 +71,8 @@
         <visual>
             <material>
-                <ambient>0.2 0.2 0.2 1</ambient>
-                <diffuse>0.2 0.2 0.2 1</diffuse>
-                <specular>0.01 0.01 0.01 1</specular>
-                <emissive>0.01 0.01 0.01 1</emissive>
+                <ambient>${ambient}</ambient>
+                <diffuse>${diffuse}</diffuse>
+                <specular>${specular}</specular>
+                <emissive>${emissive}</emissive>
             </material>
         </visual>
@@ -143,8 +146,8 @@
         <visual>
             <material>
-                <ambient>0.2 0.2 0.2 1</ambient>
-                <diffuse>0.2 0.2 0.2 1</diffuse>
-                <specular>0.01 0.01 0.01 1</specular>
-                <emissive>0.01 0.01 0.01 1</emissive>
+                <ambient>${ambient}</ambient>
+                <diffuse>${diffuse}</diffuse>
+                <specular>${specular}</specular>
+                <emissive>${emissive}</emissive>
             </material>
         </visual>
@@ -218,8 +221,8 @@
         <visual>
             <material>
-                <ambient>0.2 0.2 0.2 1</ambient>
-                <diffuse>0.2 0.2 0.2 1</diffuse>
-                <specular>0.01 0.01 0.01 1</specular>
-                <emissive>0.01 0.01 0.01 1</emissive>
+                <ambient>${ambient}</ambient>
+                <diffuse>${diffuse}</diffuse>
+                <specular>${specular}</specular>
+                <emissive>${emissive}</emissive>
             </material>
         </visual>

File: PARAM/lbr_description/urdf/Grieel/grieel_gazebo_colors.xacro (robot description, xacro)
@@ -8,4 +8,8 @@
         <xacro:include filename="$(find lbr_description)/urdf/Grieel/grieel_gripper_description.xacro" />
     </xacro:unless>
+    <xacro:property name="ambient" value="0.2 0.2 0.2 1"/>
+    <xacro:property name="diffuse" value="0.2 0.2 0.2 1"/>
+    <xacro:property name="specular" value="0.01 0.01 0.01 1"/>
+    <xacro:property name="emissive" value="0.01 0.01 0.01 1"/>
     <xacro:macro name="gazebo_colors_macro" params="prefix">
         <!-- Gazebo tag for support gripper/wheel phisical characteristics -->
@@ -30,8 +34,8 @@
             <visual>
               <material>
-                <ambient>0.2 0.2 0.2 1</ambient>
-                <diffuse>0.2 0.2 0.2 1</diffuse>
-                <specular>0.01 0.01 0.01 1</specular>
-                <emissive>0.01 0.01 0.01 1</emissive>
+                <ambient>${ambient}</ambient>
+                <diffuse>${diffuse}</diffuse>
+                <specular>${specular}</specular>
+                <emissive>${emissive}</emissive>
               </material>
             </visual>
@@ -41,8 +45,8 @@
             <visual>
               <material>
-                <ambient>0.2 0.2 0.2 1</ambient>
-                <diffuse>0.2 0.2 0.2 1</diffuse>
-                <specular>0.01 0.01 0.01 1</specular>
-                <emissive>0.01 0.01 0.01 1</emissive>
+                <ambient>${ambient}</ambient>
+                <diffuse>${diffuse}</diffuse>
+                <specular>${specular}</specular>
+                <emissive>${emissive}</emissive>
               </material>
             </visual>
@@ -52,8 +56,8 @@
             <visual>
               <material>
-                <ambient>0.2 0.2 0.2 1</ambient>
-                <diffuse>0.2 0.2 0.2 1</diffuse>
-                <specular>0.01 0.01 0.01 1</specular>
-                <emissive>0.01 0.01 0.01 1</emissive>
+                <ambient>${ambient}</ambient>
+                <diffuse>${diffuse}</diffuse>
+                <specular>${specular}</specular>
+                <emissive>${emissive}</emissive>
               </material>
             </visual>
@@ -63,8 +67,8 @@
             <visual>
               <material>
-                <ambient>0.2 0.2 0.2 1</ambient>
-                <diffuse>0.2 0.2 0.2 1</diffuse>
-                <specular>0.01 0.01 0.01 1</specular>
-                <emissive>0.01 0.01 0.01 1</emissive>
+                <ambient>${ambient}</ambient>
+                <diffuse>${diffuse}</diffuse>
+                <specular>${specular}</specular>
+                <emissive>${emissive}</emissive>
               </material>
             </visual>
@@ -74,8 +78,8 @@
             <visual>
               <material>
-                <ambient>0.2 0.2 0.2 1</ambient>
-                <diffuse>0.2 0.2 0.2 1</diffuse>
-                <specular>0.01 0.01 0.01 1</specular>
-                <emissive>0.01 0.01 0.01 1</emissive>
+                <ambient>${ambient}</ambient>
+                <diffuse>${diffuse}</diffuse>
+                <specular>${specular}</specular>
+                <emissive>${emissive}</emissive>
               </material>
             </visual>
@@ -85,8 +89,8 @@
             <visual>
               <material>
-                <ambient>0.2 0.2 0.2 1</ambient>
-                <diffuse>0.2 0.2 0.2 1</diffuse>
-                <specular>0.01 0.01 0.01 1</specular>
-                <emissive>0.01 0.01 0.01 1</emissive>
+                <ambient>${ambient}</ambient>
+                <diffuse>${diffuse}</diffuse>
+                <specular>${specular}</specular>
+                <emissive>${emissive}</emissive>
               </material>
             </visual>
@@ -96,8 +100,8 @@
             <visual>
               <material>
-                <ambient>0.2 0.2 0.2 1</ambient>
-                <diffuse>0.2 0.2 0.2 1</diffuse>
-                <specular>0.01 0.01 0.01 1</specular>
-                <emissive>0.01 0.01 0.01 1</emissive>
+                <ambient>${ambient}</ambient>
+                <diffuse>${diffuse}</diffuse>
+                <specular>${specular}</specular>
+                <emissive>${emissive}</emissive>
               </material>
             </visual>
@@ -107,8 +111,8 @@
             <visual>
               <material>
-                <ambient>0.2 0.2 0.2 1</ambient>
-                <diffuse>0.2 0.2 0.2 1</diffuse>
-                <specular>0.01 0.01 0.01 1</specular>
-                <emissive>0.01 0.01 0.01 1</emissive>
+                <ambient>${ambient}</ambient>
+                <diffuse>${diffuse}</diffuse>
+                <specular>${specular}</specular>
+                <emissive>${emissive}</emissive>
               </material>
             </visual>
@@ -140,8 +144,8 @@
             <visual>
               <material>
-                <ambient>0.2 0.2 0.2 1</ambient>
-                <diffuse>0.2 0.2 0.2 1</diffuse>
-                <specular>0.01 0.01 0.01 1</specular>
-                <emissive>0.01 0.01 0.01 1</emissive>
+                <ambient>${ambient}</ambient>
+                <diffuse>${diffuse}</diffuse>
+                <specular>${specular}</specular>
+                <emissive>${emissive}</emissive>
               </material>
             </visual>

File: PARAM/lbr_description/urdf/Grieel/grieel_gazebo_ros2_control.xacro (robot description, xacro)
@@ -6,4 +6,5 @@
                 <parameters>$(find lbr_description)/config/grieel_controllers.yaml</parameters>
                 <ros>
+                    <parameter name="use_sim_time" type="bool">true</parameter>
                     <remapping>/controller_manager/robot_description:=/robot_description</remapping>
                 </ros>

File: PARAM/lbr_description/urdf/Grieel/grieel_gripper_splitted.xacro (robot description, xacro)
@@ -3,12 +3,12 @@
      Commit Version: 1.6.0-4-g7f85cfe  Build Version: 1.6.7995.38578
      For more information, please see http://wiki.ros.org/sw_urdf_exporter -->
-<robot
-  name="assembled_gripper_mode" xmlns:xacro="http://ros.org/wiki/xacro">
+<robot name="assembled_gripper_mode" xmlns:xacro="http://ros.org/wiki/xacro">
   <xacro:macro name="grieel_hand_macro" params="prefix">
   <xacro:include filename="$(find lbr_description)/urdf/Grieel/grieel_finger_macro.xacro" />
   <xacro:include filename="$(find lbr_description)/urdf/Grieel/grieel_first_finger_macro.xacro" />
+  <xacro:include filename="$(find lbr_description)/urdf/Grieel/grieel_gripper_description.xacro" />
     <joint
         name="${prefix}_driving"
-        type="continuous">
+        type="revolute">
         <origin
         xyz="0.0131 0 0.04576"
@@ -21,6 +21,8 @@
         xyz="1 0 0" />
         <limit
-        effort="0.0"
-        velocity="0.0" />
+        lower="1E14"
+        upper="-1E14"
+        effort="10.0"
+        velocity="10.0" />
         <dynamics damping="0.1" friction="0.4"/>
     </joint>

File: PARAM/lbr_description/urdf/Grieel/grieel_ros2_control.xacro (robot description, xacro)
@@ -6,4 +6,107 @@
         <plugin>gz_ros2_control/GazeboSimSystem</plugin>
       </hardware>
+      <!-- LIMB JOINTS -->
+      <joint name="${prefix}_B2C">
+        <command_interface name="position">
+                    <param name="min">-2.10</param>
+                    <param name="max">2.10</param>
+        </command_interface>
+        <command_interface name="effort">
+          <param name="min">-10</param>
+          <param name="max">10</param>
+        </command_interface>
+        <state_interface name="position">
+            <param name="initial_value">0.0</param>
+        </state_interface>
+        <state_interface name="velocity"/>
+      </joint>
+      <joint name="${prefix}_C2F">
+        <command_interface name="position">
+                    <param name="min">-1.95</param>
+                    <param name="max">1.3</param>
+        </command_interface>
+        <command_interface name="effort">
+          <param name="min">-10</param>
+          <param name="max">10</param>
+        </command_interface>
+        <state_interface name="position">
+            <param name="initial_value">0.0</param>
+        </state_interface>
+        <state_interface name="velocity"/>
+      </joint>
+      <joint name="${prefix}_F2T">
+        <command_interface name="effort">
+          <param name="min">-10</param>
+          <param name="max">10</param>
+        </command_interface>
+        <command_interface name="position">
+                    <param name="min">-0.4</param>
+                    <param name="max">2.95</param>
+        </command_interface>
+        <state_interface name="position">
+            <param name="initial_value">1.5707963267948966</param>
+        </state_interface>
+        <state_interface name="velocity"/>
+      </joint>
+      <joint name="${prefix}_T2E">
+        <command_interface name="position">
+                    <param name="min">-1.57</param>
+                    <param name="max">1.57</param>
+        </command_interface>
+        <command_interface name="effort">
+          <param name="min">-10</param>
+          <param name="max">10</param>
+        </command_interface>
+        <state_interface name="position">
+            <param name="initial_value">0.0</param>
+        </state_interface>
+        <state_interface name="velocity"/>
+      </joint>
+      <joint name="${prefix}_wristH">
+        <command_interface name="position">
+                    <param name="min">-3.14159265358</param>
+                    <param name="max">3.14159265358</param>
+        </command_interface>
+        <command_interface name="effort">
+          <param name="min">-10</param>
+          <param name="max">10</param>
+        </command_interface>
+        <state_interface name="position">
+            <param name="initial_value">0.0</param>
+        </state_interface>
+        <state_interface name="velocity"/>
+      </joint>
+      <joint name="${prefix}_wristV">
+        <command_interface name="position">
+                    <param name="min">-0.78539816339</param>
+                    <param name="max">1.57079632679</param>
+        </command_interface>
+        <command_interface name="effort">
+          <param name="min">-10</param>
+          <param name="max">10</param>
+        </command_interface>
+        <state_interface name="position">
+            <param name="initial_value">0.0</param>
+        </state_interface>
+        <state_interface name="velocity"/>
+      </joint>
+      <joint name="${prefix}_driving">
+        <command_interface name="position"/>
+        <command_interface name="velocity">
+                    <param name="min">-5</param>
+                    <param name="max">5</param>
+        </command_interface>
+        <command_interface name="effort">
+          <param name="min">-10</param>
+          <param name="max">10</param>
+        </command_interface>
+        <state_interface name="position">
+            <param name="initial_value">0.0</param>
+        </state_interface>
+        <state_interface name="velocity">
+            <param name="initial_value">0.0</param>
+        </state_interface>
+      </joint>
+      <!-- GRIPPER JOINTS (FINGERS) -->
       <joint name="${prefix}_F1_H2P1">
         <command_interface name="position">

File: PARAM/lbr_description/urdf/Grieel/lbr_base_description.xacro (robot description, xacro)
@@ -6,4 +6,8 @@
   name="LIMBERO_v1_8_Base" xmlns:xacro="http://ros.org/wiki/xacro">
   <xacro:macro name="base_macro">
+  <xacro:property name="ambient" value="0.2 0.2 0.2 1"/>
+  <xacro:property name="diffuse" value="0.2 0.2 0.2 1"/>
+  <xacro:property name="specular" value="0.01 0.01 0.01 1"/>
+  <xacro:property name="emissive" value="0.01 0.01 0.01 1"/>
     <link
       name="base_link">
@@ -50,10 +54,14 @@
       <visual>
         <material>
-          <ambient>0.2 0.2 0.2 1</ambient>
-          <diffuse>0.2 0.2 0.2 1</diffuse>
-          <specular>0.01 0.01 0.01 1</specular>
-          <emissive>0.01 0.01 0.01 1</emissive>
+            <ambient>${ambient}</ambient>
+            <diffuse>${diffuse}</diffuse>
+            <specular>${specular}</specular>
+            <emissive>${emissive}</emissive>
         </material>
       </visual>
+      <mu1>1.0</mu1>
+      <mu2>1.0</mu2>
+      <kp>1000000</kp>
+      <kd>1.0</kd>
     </gazebo>
 <!--
