Commit message: simple inertia and collision to simplify simulation

File: PARAM/lbr_description/urdf/Grieel/grieel_finger_macro.xacro (robot description, xacro)
@@ -5,4 +5,5 @@
 <robot
   name="assembled_gripper_mode" xmlns:xacro="http://ros.org/wiki/xacro">
+  <xacro:include filename="$(find lbr_description)/urdf/Grieel/inertial_macro.xacro" />
   <xacro:arg name="not_first_finger" default="false" />
   <xacro:property name="ambient" value="0.2 0.2 0.2 1"/>
@@ -31,5 +32,5 @@
     <link
         name="${prefix}_${name}_phalanx1">
-        <inertial>
+        <!-- <inertial>
             <origin
                 xyz="0.00162585 0.00031929 0.01672194"
@@ -44,5 +45,8 @@
                 iyz="-4.29494199e-09"
                 izz="8.86398503e-08" />
-        </inertial>
+        </inertial> -->
+        <xacro:inertial_box mass="0.003797793442763989" x="0.017" y="0.018" z="0.038">
+            <origin xyz="0.00162585 0.00031929 0.019" rpy="0 0 0"/>
+        </xacro:inertial_box>
         <visual>
         <origin
@@ -61,9 +65,10 @@
         <collision>
         <origin
-            xyz="0 0 0"
-            rpy="0 0 0" />
-        <geometry>
-            <mesh
-            filename="file://$(find lbr_description)/meshes/Grieel_gripper_mode/gripper_Link_finger1.stl" />
+            xyz="0 0 0.019"
+            rpy="0 0 0" />
+        <geometry>
+            <!-- <mesh
+            filename="file://$(find lbr_description)/meshes/Grieel_gripper_mode/gripper_Link_finger1.stl" /> -->
+            <box size="0.017 0.018 0.038" />
         </geometry>
         </collision>
@@ -79,6 +84,6 @@
             </material>
         </visual>
-        <mu1>1.0</mu1>
-        <mu2>1.0</mu2>
+        <mu1>1.5</mu1>
+        <mu2>1.5</mu2>
         <kp>1000000</kp>
         <kd>1.0</kd>
@@ -106,5 +111,5 @@
     <link
         name="${prefix}_${name}_phalanx2">
-        <inertial>
+        <!-- <inertial>
             <origin
                 xyz="-0.00673704 0.00047222 0.01186178"
@@ -119,5 +124,8 @@
                 iyz="7.23067218e-09"
                 izz="2.30350901e-06" />
-        </inertial>
+        </inertial> -->
+        <xacro:inertial_box mass="0.013082859723205855" x="0.017" y="0.04" z="0.036">
+            <origin xyz="-0.00673704 0.00047222 0.018" rpy="0 0 0"/>
+        </xacro:inertial_box>
         <visual>
         <origin
@@ -136,9 +144,10 @@
         <collision>
         <origin
-            xyz="0 0 0"
-            rpy="0 0 0" />
-        <geometry>
-            <mesh
-            filename="file://$(find lbr_description)/meshes/Grieel_gripper_mode/gripper_Link_finger2.stl" />
+            xyz="0 0 0.018"
+            rpy="0 0 0" />
+        <geometry>
+            <!-- <mesh
+            filename="file://$(find lbr_description)/meshes/Grieel_gripper_mode/gripper_Link_finger2.stl" /> -->
+            <box size="0.017 0.04 0.036" />
         </geometry>
         </collision>
@@ -154,6 +163,6 @@
             </material>
         </visual>
-        <mu1>1.0</mu1>
-        <mu2>1.0</mu2>
+        <mu1>1.5</mu1>
+        <mu2>1.5</mu2>
         <kp>1000000</kp>
         <kd>1.0</kd>
@@ -181,5 +190,5 @@
     <link
         name="${prefix}_${name}_phalanx3">
-        <inertial>
+        <!-- <inertial>
             <origin
                 xyz="-0.00232913 0.00061377 0.01268651"
@@ -194,5 +203,8 @@
                 iyz="1.69572891e-09"
                 izz="4.48441736e-08" />
-        </inertial>
+        </inertial> -->
+        <xacro:inertial_box mass="0.0024217622661742476" x="0.017" y="0.012" z="0.028">
+            <origin xyz="-0.00232913 0.00061377 0.014" rpy="0 0 0"/>
+        </xacro:inertial_box>
         <visual>
         <origin
@@ -211,9 +223,10 @@
         <collision>
         <origin
-            xyz="0 0 0"
-            rpy="0 0 0" />
-        <geometry>
-            <mesh
-            filename="file://$(find lbr_description)/meshes/Grieel_gripper_mode/gripper_Link_finger3.stl" />
+            xyz="0 0 0.014"
+            rpy="0 0 0" />
+        <geometry>
+            <!-- <mesh
+            filename="file://$(find lbr_description)/meshes/Grieel_gripper_mode/gripper_Link_finger3.stl" /> -->
+            <box size="0.017 0.012 0.028" />
         </geometry>
         </collision>
@@ -229,6 +242,6 @@
             </material>
         </visual>
-        <mu1>1.0</mu1>
-        <mu2>1.0</mu2>
+        <mu1>1.5</mu1>
+        <mu2>1.5</mu2>
         <kp>1000000</kp>
         <kd>1.0</kd>

File: PARAM/lbr_description/urdf/Grieel/grieel_first_finger_macro.xacro (robot description, xacro)
@@ -5,4 +5,5 @@
 <robot
   name="assembled_gripper_mode" xmlns:xacro="http://ros.org/wiki/xacro">
+  <xacro:include filename="$(find lbr_description)/urdf/Grieel/inertial_macro.xacro" />
   <xacro:property name="ambient" value="0.2 0.2 0.2 1"/>
   <xacro:property name="diffuse" value="0.2 0.2 0.2 1"/>
@@ -29,5 +30,5 @@
     <link
         name="${prefix}_${name}_phalanx1">
-        <inertial>
+        <!-- <inertial>
             <origin
                 xyz="0.00162585 0.00031929 0.01672194"
@@ -42,5 +43,8 @@
                 iyz="-4.29494199e-09"
                 izz="8.86398503e-08" />
-        </inertial>
+        </inertial> -->
+        <xacro:inertial_box mass="0.003797793442763989" x="0.017" y="0.018" z="0.038">
+            <origin xyz="0.00162585 0.00031929 0.019" rpy="0 0 0"/>
+        </xacro:inertial_box>
         <visual>
         <origin
@@ -59,9 +63,10 @@
         <collision>
         <origin
-            xyz="0 0 0"
-            rpy="0 0 0" />
-        <geometry>
-            <mesh
-            filename="file://$(find lbr_description)/meshes/Grieel_gripper_mode/gripper_Link_finger1.stl" />
+            xyz="0 0 0.019"
+            rpy="0 0 0" />
+        <geometry>
+            <!-- <mesh
+            filename="file://$(find lbr_description)/meshes/Grieel_gripper_mode/gripper_Link_finger1.stl" /> -->
+            <box size="0.017 0.018 0.038" />
         </geometry>
         </collision>
@@ -77,6 +82,6 @@
             </material>
         </visual>
-        <mu1>1.0</mu1>
-        <mu2>1.0</mu2>
+        <mu1>1.5</mu1>
+        <mu2>1.5</mu2>
         <kp>1000000</kp>
         <kd>1.0</kd>
@@ -104,5 +109,5 @@
     <link
         name="${prefix}_${name}_phalanx2">
-        <inertial>
+        <!-- <inertial>
             <origin
                 xyz="-0.00673704 0.00047222 0.01186178"
@@ -117,5 +122,8 @@
                 iyz="7.23067218e-09"
                 izz="2.30350901e-06" />
-        </inertial>
+        </inertial> -->
+        <xacro:inertial_box mass="0.013082859723205855" x="0.017" y="0.04" z="0.036">
+            <origin xyz="-0.00673704 0.00047222 0.018" rpy="0 0 0"/>
+        </xacro:inertial_box>
         <visual>
         <origin
@@ -134,9 +142,10 @@
         <collision>
         <origin
-            xyz="0 0 0"
-            rpy="0 0 0" />
-        <geometry>
-            <mesh
-            filename="file://$(find lbr_description)/meshes/Grieel_gripper_mode/gripper_Link_finger2.stl" />
+            xyz="0 0 0.018"
+            rpy="0 0 0" />
+        <geometry>
+            <!-- <mesh
+            filename="file://$(find lbr_description)/meshes/Grieel_gripper_mode/gripper_Link_finger2.stl" /> -->
+            <box size="0.017 0.04 0.036" />
         </geometry>
         </collision>
@@ -152,6 +161,6 @@
             </material>
         </visual>
-        <mu1>1.0</mu1>
-        <mu2>1.0</mu2>
+        <mu1>1.5</mu1>
+        <mu2>1.5</mu2>
         <kp>1000000</kp>
         <kd>1.0</kd>
@@ -179,5 +188,5 @@
     <link
         name="${prefix}_${name}_phalanx3">
-        <inertial>
+        <!-- <inertial>
             <origin
                 xyz="-0.00232913 0.00061377 0.01268651"
@@ -192,5 +201,8 @@
                 iyz="1.69572891e-09"
                 izz="4.48441736e-08" />
-        </inertial>
+        </inertial> -->
+        <xacro:inertial_box mass="0.0024217622661742476" x="0.017" y="0.012" z="0.028">
+            <origin xyz="-0.00232913 0.00061377 0.014" rpy="0 0 0"/>
+        </xacro:inertial_box>
         <visual>
         <origin
@@ -209,9 +221,10 @@
         <collision>
         <origin
-            xyz="0 0 0"
-            rpy="0 0 0" />
-        <geometry>
-            <mesh
-            filename="file://$(find lbr_description)/meshes/Grieel_gripper_mode/gripper_Link_finger3.stl" />
+            xyz="0 0 0.014"
+            rpy="0 0 0" />
+        <geometry>
+            <!-- <mesh
+            filename="file://$(find lbr_description)/meshes/Grieel_gripper_mode/gripper_Link_finger3.stl" /> -->
+            <box size="0.017 0.012 0.028" />
         </geometry>
         </collision>
@@ -227,6 +240,6 @@
             </material>
         </visual>
-        <mu1>1.0</mu1>
-        <mu2>1.0</mu2>
+        <mu1>1.5</mu1>
+        <mu2>1.5</mu2>
         <kp>1000000</kp>
         <kd>1.0</kd>

File: PARAM/lbr_description/urdf/Grieel/grieel_gripper_description.xacro (robot description, xacro)
@@ -6,5 +6,6 @@
   name="assembled_gripper_mode" xmlns:xacro="http://ros.org/wiki/xacro">
   <xacro:macro name="grieel_gripper_macro" params="prefix parent">
-  <xacro:include filename="$(find lbr_description)/urdf/Grieel/grieel_gripper_splitted.xacro" />
+    <xacro:include filename="$(find lbr_description)/urdf/Grieel/grieel_gripper_splitted.xacro" />
+    <xacro:include filename="$(find lbr_description)/urdf/Grieel/inertial_macro.xacro" />
     <xacro:property name="friction" value="0.1"/>
     <xacro:property name="damping" value="0.05"/>
@@ -69,5 +70,5 @@
   <link
     name="${prefix}_wristV_Link">
-    <inertial>
+    <!-- <inertial>
       <origin
         xyz="0.0214166502499745 0.000471129500725836 0.0113219457469963"
@@ -82,5 +83,8 @@
         iyz="-1.3142285327366E-09"
         izz="1.79824315026287E-05" />
-    </inertial>
+    </inertial> -->
+    <xacro:inertial_box mass="0.102059813857681" x="0.0489" y="0.0489" z="0.0465">
+            <origin xyz="${0.020217+0.0214166502499745} 0.000471129500725836 ${0.011897+0.0113219457469963}" rpy="0 0 0"/>
+    </xacro:inertial_box>
     <visual>
       <origin
@@ -99,9 +103,10 @@
     <collision>
       <origin
-        xyz="0 0 0"
-        rpy="0 0 0" />
-      <geometry>
-        <mesh
-          filename="file://$(find lbr_description)/meshes/Grieel_gripper_mode/wristV_Link.STL" />
+        xyz="0.020217 0 0.011897"
+        rpy="0 0 0" />
+      <geometry>
+        <!-- <mesh
+          filename="file://$(find lbr_description)/meshes/Grieel_gripper_mode/wristV_Link.STL" /> -->
+            <box size="0.0489 0.0489 0.0465" />
       </geometry>
     </collision>
@@ -128,5 +133,5 @@
   <link
     name="${prefix}_driving_Link">
-    <inertial>
+    <!-- <inertial>
       <origin
         xyz="5.44808065291863E-05 0.00431293338596027 0.0448909989385787"
@@ -141,5 +146,8 @@
         iyz="4.14273177876885E-09"
         izz="4.32511275712205E-05" />
-    </inertial>
+    </inertial> -->
+    <xacro:inertial_box mass="0.132659951311712" x="0.0585" y="0.0595" z="0.0354">
+            <origin xyz="5.44808065291863E-05 0.00431293338596027 ${0.040724+0.0448909989385787}" rpy="0 0 0"/>
+    </xacro:inertial_box>
     <visual>
       <origin
@@ -158,9 +166,10 @@
     <collision>
       <origin
-        xyz="0 0 0"
-        rpy="0 0 0" />
-      <geometry>
-        <mesh
-          filename="file://$(find lbr_description)/meshes/Grieel_gripper_mode/driving_Link.STL" />
+        xyz="0 0 0.040724"
+        rpy="0 0 0" />
+      <geometry>
+        <!-- <mesh
+          filename="file://$(find lbr_description)/meshes/Grieel_gripper_mode/driving_Link.STL" /> -->
+            <box size="0.0585 0.0595 0.0354" />
       </geometry>
     </collision>

File: PARAM/lbr_description/urdf/Grieel/grieel_gripper_splitted.xacro (robot description, xacro)
@@ -8,4 +8,5 @@
   <xacro:include filename="$(find lbr_description)/urdf/Grieel/grieel_first_finger_macro.xacro" />
   <xacro:include filename="$(find lbr_description)/urdf/Grieel/grieel_gripper_description.xacro" />
+  <xacro:include filename="$(find lbr_description)/urdf/Grieel/inertial_macro.xacro" />
     <joint
         name="${prefix}_driving"
@@ -29,5 +30,5 @@
     <link
         name="${prefix}_hand_Link">
-        <inertial>
+        <!-- <inertial>
         <origin
             xyz="0.05982052 -0.00756175 0.00448521"
@@ -42,5 +43,8 @@
             iyz="-2.56859397e-06"
             izz="1.13275414e-04" />
-        </inertial>
+        </inertial> -->
+        <xacro:inertial_box mass="0.125" x="0.06" y="0.04" z="0.04">
+            <origin xyz="${0.05982052+0.065} -0.00756175 0.00448521" rpy="0 0 0"/>
+        </xacro:inertial_box>
         <visual>
         <origin
@@ -59,9 +63,10 @@
         <collision name="${prefix}_gripper_Link_collision">
         <origin
-            xyz="0 0 0"
+            xyz="0.065 0 0"
             rpy="0 0 0" />
         <geometry>
-            <mesh
-            filename="file://$(find lbr_description)/meshes/Grieel_gripper_mode/gripper_Link_Hand.stl" />
+            <!-- <mesh
+            filename="file://$(find lbr_description)/meshes/Grieel_gripper_mode/gripper_Link_Hand.stl" /> -->
+            <box size="0.06 0.04 0.04" />
         </geometry>
         </collision>

File: PARAM/lbr_description/urdf/Grieel/lbr_base_description.xacro (robot description, xacro)
@@ -6,4 +6,5 @@
   name="LIMBERO_v1_8_Base" xmlns:xacro="http://ros.org/wiki/xacro">
   <xacro:macro name="base_macro">
+  <xacro:include filename="$(find lbr_description)/urdf/Grieel/inertial_macro.xacro" />
   <xacro:property name="ambient" value="0.2 0.2 0.2 1"/>
   <xacro:property name="diffuse" value="0.2 0.2 0.2 1"/>
@@ -12,5 +13,5 @@
     <link
       name="base_link">
-      <inertial>
+      <!-- <inertial>
         <origin
           xyz="0 0 -0.0030083"
@@ -25,5 +26,8 @@
           iyz="-1.4424E-06"
           izz="0.0034682" />
-      </inertial>
+      </inertial> -->
+      <xacro:inertial_box mass="3.1152" x="0.24" y="0.24" z="0.16">
+            <origin xyz="0 0 -0.0030083" rpy="0 0 0"/>
+      </xacro:inertial_box>
       <visual>
         <origin
@@ -45,6 +49,7 @@
           rpy="0 0 0" />
         <geometry>
-          <mesh
-            filename="file://$(find lbr_description)/meshes/base.STL" scale="1.0 1.0 1.0"/>
+          <!-- <mesh
+            filename="file://$(find lbr_description)/meshes/base.STL" scale="1.0 1.0 1.0"/> -->
+            <box size="0.24 0.24 0.16" />
         </geometry>
       </collision>

File: PARAM/lbr_description/urdf/Grieel/lbr_limb_description.xacro (robot description, xacro)
@@ -6,4 +6,5 @@
   name="LIMBERO_v1_7_Limb" xmlns:xacro="http://ros.org/wiki/xacro">
   <xacro:macro name="limb_macro" params="prefix parent radius">
+    <xacro:include filename="$(find lbr_description)/urdf/Grieel/inertial_macro.xacro" />
     <xacro:property name="friction" value="0.1"/>
     <xacro:property name="damping" value="0.05"/>
@@ -21,5 +22,5 @@
     <link
       name="${prefix}_limb_root">
-      <inertial>
+      <!-- <inertial>
         <origin
           xyz="-0.015029 -7.7571E-11 -0.047318"
@@ -34,5 +35,8 @@
           iyz="-8.2973E-14"
           izz="3.1728E-05" />
-      </inertial>
+      </inertial> -->
+      <xacro:inertial_box mass="0.08459" x="0.0585" y="0.0335" z="0.0543">
+            <origin xyz="${-0.015029+0.02925} -7.7571E-11 ${-0.047318-0.047551}" rpy="0 0 0"/>
+      </xacro:inertial_box>
       <visual>
         <origin
@@ -51,9 +55,10 @@
       <collision>
         <origin
-          xyz="0 0 0"
-          rpy="0 0 0" />
-        <geometry>
-          <mesh
-            filename="file://$(find lbr_description)/meshes/limb_root.STL" />
+          xyz="0.02925 0 -0.047551"
+          rpy="0 0 0" />
+        <geometry>
+          <!-- <mesh
+            filename="file://$(find lbr_description)/meshes/limb_root.STL" /> -->
+            <box size="0.0585 0.0335 0.0543" />
         </geometry>
       </collision>
@@ -61,5 +66,5 @@
     <link
       name="${prefix}_coxa">
-      <inertial>
+      <!-- <inertial>
         <origin
           xyz="0.015938 0.00063302 -0.0015013"
@@ -74,5 +79,8 @@
           iyz="8.2973E-14"
           izz="4.2122E-05" />
-      </inertial>
+      </inertial> -->
+      <xacro:inertial_box mass="0.09109" x="0.0585" y="0.0543" z="0.0402">
+            <origin xyz="${0.015938+0.017478} 0.00063302 -0.0015013" rpy="0 0 0"/>
+      </xacro:inertial_box>
       <visual>
         <origin
@@ -91,9 +99,10 @@
       <collision>
         <origin
-          xyz="0 0 0"
-          rpy="0 0 0" />
-        <geometry>
-          <mesh
-            filename="file://$(find lbr_description)/meshes/coxa.STL" />
+          xyz="0.017478 0 0"
+          rpy="0 0 0" />
+        <geometry>
+          <!-- <mesh
+            filename="file://$(find lbr_description)/meshes/coxa.STL" /> -->
+            <box size="0.0585 0.0543 0.0402" />
         </geometry>
       </collision>
@@ -130,5 +139,5 @@
     <link
       name="${prefix}_femur">
-      <inertial>
+      <!-- <inertial>
         <origin
           xyz="0.10083 0.00014739 -3.217E-08"
@@ -143,5 +152,8 @@
           iyz="2.5988E-11"
           izz="4.8164E-05" />
-      </inertial>
+      </inertial> -->
+      <xacro:inertial_cylinder mass="0.12821" length="0.177" radius="0.013">
+            <origin xyz="${0.10083+0.11} 0.00014739 -3.217E-08" rpy="0 1.57079632679489661923 0"/>
+      </xacro:inertial_cylinder>
       <visual>
         <origin
@@ -160,9 +172,10 @@
       <collision>
         <origin
-          xyz="0 0 0"
-          rpy="0 0 0" />
-        <geometry>
-          <mesh
-            filename="file://$(find lbr_description)/meshes/femur.STL" />
+          xyz="0.11 0 0"
+          rpy="0 1.57079632679489661923 0" />
+        <geometry>
+          <!-- <mesh
+            filename="file://$(find lbr_description)/meshes/femur.STL" /> -->
+            <cylinder radius="0.013" length="0.177"/>
         </geometry>
       </collision>
@@ -199,5 +212,5 @@
     <link
       name="${prefix}_tibia">
-      <inertial>
+      <!-- <inertial>
         <origin
           xyz="0.10298 1.1638E-07 0.019231"
@@ -212,5 +225,8 @@
           iyz="2.414E-08"
           izz="2.8843E-05" />
-      </inertial>
+      </inertial> -->
+      <xacro:inertial_cylinder mass="0.061841" length="0.14" radius="0.01">
+            <origin xyz="${0.10298+0.08} 1.1638E-07 ${0.019231+0.027}" rpy="0 1.78023583703421616846 0"/>
+      </xacro:inertial_cylinder>
       <visual>
         <origin
@@ -229,9 +245,10 @@
       <collision>
         <origin
-          xyz="0 0 0"
-          rpy="0 0 0" />
-        <geometry>
-          <mesh
-            filename="file://$(find lbr_description)/meshes/tibia.STL" />
+          xyz="0.08 0 0.027"
+          rpy="0 1.78023583703421616846 0" />
+        <geometry>
+          <!-- <mesh
+            filename="file://$(find lbr_description)/meshes/tibia.STL" /> -->
+                <cylinder radius="0.01" length="0.14"/>
         </geometry>
       </collision>
@@ -269,5 +286,5 @@
     <link
       name="${prefix}_limb_end">
-      <inertial>
+      <!-- <inertial>
         <origin
           xyz="-0.011645 0.00042918 -9.53E-12"
@@ -282,5 +299,8 @@
           iyz="-3.9438E-17"
           izz="2.2308E-05" />
-      </inertial>
+      </inertial> -->
+      <xacro:inertial_box mass="0.081999" x="0.0465" y="0.04245" z="0.0285">
+            <origin xyz="${-0.011645-0.010236} 0.00042918 -9.53E-12" rpy="0 0 0"/>
+      </xacro:inertial_box>
       <visual>
         <origin
@@ -299,9 +319,10 @@
       <collision>
         <origin
-          xyz="0 0 0"
-          rpy="0 0 0" />
-        <geometry>
-          <mesh
-            filename="file://$(find lbr_description)/meshes/limb_end.STL" />
+          xyz="-0.010236 0 0"
+          rpy="0 0 0" />
+        <geometry>
+          <!-- <mesh
+            filename="file://$(find lbr_description)/meshes/limb_end.STL" /> -->
+            <box size="0.0465 0.0424 0.0285" />
         </geometry>
       </collision>
