Commit message: updating simulation

File: PARAM/lbr_description/urdf/Grieel/grieel_finger_macro.xacro (robot description, xacro)
@@ -7,8 +7,8 @@
   <xacro:include filename="$(find lbr_description)/urdf/Grieel/inertial_macro.xacro" />
   <xacro:arg name="not_first_finger" default="false" />
-  <xacro:property name="ambient" value="0.2 0.2 0.2 1"/>
+  <xacro:property name="ambient" value="0.1 0.1 0.1 1"/>
   <xacro:property name="diffuse" value="0.2 0.2 0.2 1"/>
-  <xacro:property name="specular" value="0.01 0.01 0.01 1"/>
-  <xacro:property name="emissive" value="0.01 0.01 0.01 1"/>
+  <xacro:property name="specular" value="0.4 0.4 0.4 1"/>
+  <xacro:property name="emissive" value="0 0 0 1"/>
   <xacro:arg name="simplified" default="false" />
   <xacro:macro name="grieel_gripper_finger_macro" params="prefix name *origin">

File: PARAM/lbr_description/urdf/Grieel/grieel_first_finger_macro.xacro (robot description, xacro)
@@ -6,8 +6,8 @@
   name="assembled_gripper_mode" xmlns:xacro="http://ros.org/wiki/xacro">
   <xacro:include filename="$(find lbr_description)/urdf/Grieel/inertial_macro.xacro" />
-  <xacro:property name="ambient" value="0.2 0.2 0.2 1"/>
+  <xacro:property name="ambient" value="0.1 0.1 0.1 1"/>
   <xacro:property name="diffuse" value="0.2 0.2 0.2 1"/>
-  <xacro:property name="specular" value="0.01 0.01 0.01 1"/>
-  <xacro:property name="emissive" value="0.01 0.01 0.01 1"/>
+  <xacro:property name="specular" value="0.4 0.4 0.4 1"/>
+  <xacro:property name="emissive" value="0 0 0 1"/>
   <xacro:arg name="simplified" default="false" />
   <xacro:macro name="grieel_gripper_first_finger_macro" params="prefix name *origin">

File: PARAM/lbr_description/urdf/Grieel/grieel_gazebo_colors.xacro (robot description, xacro)
@@ -9,7 +9,7 @@
     </xacro:unless>
     <xacro:property name="ambient" value="0.2 0.2 0.2 1"/>
-    <xacro:property name="diffuse" value="0.2 0.2 0.2 1"/>
-    <xacro:property name="specular" value="0.01 0.01 0.01 1"/>
-    <xacro:property name="emissive" value="0.01 0.01 0.01 1"/>
+    <xacro:property name="diffuse" value="0.35 0.35 0.35 1"/>
+    <xacro:property name="specular" value="0.4 0.4 0.4 1"/>
+    <xacro:property name="emissive" value="0 0 0 1"/>
     <xacro:macro name="gazebo_colors_macro" params="prefix">
         <!-- Gazebo tag for support gripper/wheel phisical characteristics -->

File: PARAM/lbr_description/urdf/Grieel/grieel_gripper_description.xacro (robot description, xacro)
@@ -8,6 +8,6 @@
     <xacro:include filename="$(find lbr_description)/urdf/Grieel/grieel_gripper_splitted.xacro" />
     <xacro:include filename="$(find lbr_description)/urdf/Grieel/inertial_macro.xacro" />
-    <xacro:property name="friction" value="0.1"/>
-    <xacro:property name="damping" value="0.05"/>
+    <xacro:property name="friction" value="0.4"/>
+    <xacro:property name="damping" value="0.15"/>
     <xacro:arg name="simplified" default="false" />
     <joint

File: PARAM/lbr_description/urdf/Grieel/lbr_base_description.xacro (robot description, xacro)
@@ -8,7 +8,7 @@
   <xacro:include filename="$(find lbr_description)/urdf/Grieel/inertial_macro.xacro" />
   <xacro:property name="ambient" value="0.2 0.2 0.2 1"/>
-  <xacro:property name="diffuse" value="0.2 0.2 0.2 1"/>
-  <xacro:property name="specular" value="0.01 0.01 0.01 1"/>
-  <xacro:property name="emissive" value="0.01 0.01 0.01 1"/>
+  <xacro:property name="diffuse" value="0.35 0.35 0.35 1"/>
+  <xacro:property name="specular" value="0.4 0.4 0.4 1"/>
+  <xacro:property name="emissive" value="0 0 0 1"/>
   <xacro:arg name="simplified" default="false" />
     <link

File: PARAM/lbr_description/urdf/Grieel/lbr_limb_description.xacro (robot description, xacro)
@@ -7,6 +7,6 @@
   <xacro:macro name="limb_macro" params="prefix parent radius">
     <xacro:include filename="$(find lbr_description)/urdf/Grieel/inertial_macro.xacro" />
-    <xacro:property name="friction" value="0.1"/>
-    <xacro:property name="damping" value="0.05"/>
+    <xacro:property name="friction" value="0.4"/>
+    <xacro:property name="damping" value="0.15"/>
     <xacro:arg name="simplified" default="false" />
     <joint
