Commit message: minor description changes

File: PARAM/lbr_description/urdf/Grieel/grieel_finger_macro.xacro (robot description, xacro)
@@ -7,8 +7,4 @@
   <xacro:include filename="$(find lbr_description)/urdf/Grieel/inertial_macro.xacro" />
   <xacro:arg name="not_first_finger" default="false" />
-  <xacro:property name="ambient" value="0.1 0.1 0.1 1"/>
-  <xacro:property name="diffuse" value="0.2 0.2 0.2 1"/>
-  <xacro:property name="specular" value="0.4 0.4 0.4 1"/>
-  <xacro:property name="emissive" value="0 0 0 1"/>
   <xacro:arg name="simplified" default="false" />
   <xacro:macro name="grieel_gripper_finger_macro" params="prefix name *origin">
@@ -99,19 +95,4 @@
         </xacro:unless>
     </link>
-    <gazebo reference="${prefix}_${name}_phalanx1">
-        <material>Gazebo/Black</material>
-        <visual>
-            <material>
-                <ambient>${ambient}</ambient>
-                <diffuse>${diffuse}</diffuse>
-                <specular>${specular}</specular>
-                <emissive>${emissive}</emissive>
-            </material>
-        </visual>
-        <mu1>1.5</mu1>
-        <mu2>1.5</mu2>
-        <kp>1000000</kp>
-        <kd>1.0</kd>
-    </gazebo>
     <joint
         name="${prefix}_${name}_P12P2"
@@ -202,19 +183,4 @@
         </xacro:unless>
     </link>
-    <gazebo reference="${prefix}_${name}_phalanx2">
-        <material>Gazebo/Black</material>
-        <visual>
-            <material>
-                <ambient>${ambient}</ambient>
-                <diffuse>${diffuse}</diffuse>
-                <specular>${specular}</specular>
-                <emissive>${emissive}</emissive>
-            </material>
-        </visual>
-        <mu1>1.5</mu1>
-        <mu2>1.5</mu2>
-        <kp>1000000</kp>
-        <kd>1.0</kd>
-    </gazebo>
    <joint
         name="${prefix}_${name}_P22P3"
@@ -308,19 +274,4 @@
         </xacro:unless>
     </link>
-    <gazebo reference="${prefix}_${name}_phalanx3">
-        <material>Gazebo/Black</material>
-        <visual>
-            <material>
-                <ambient>${ambient}</ambient>
-                <diffuse>${diffuse}</diffuse>
-                <specular>${specular}</specular>
-                <emissive>${emissive}</emissive>
-            </material>
-        </visual>
-        <mu1>1.5</mu1>
-        <mu2>1.5</mu2>
-        <kp>1000000</kp>
-        <kd>1.0</kd>
-    </gazebo>
   </xacro:macro>
 </robot>

File: PARAM/lbr_description/urdf/Grieel/grieel_first_finger_macro.xacro (robot description, xacro)
@@ -6,8 +6,4 @@
   name="assembled_gripper_mode" xmlns:xacro="http://ros.org/wiki/xacro">
   <xacro:include filename="$(find lbr_description)/urdf/Grieel/inertial_macro.xacro" />
-  <xacro:property name="ambient" value="0.1 0.1 0.1 1"/>
-  <xacro:property name="diffuse" value="0.2 0.2 0.2 1"/>
-  <xacro:property name="specular" value="0.4 0.4 0.4 1"/>
-  <xacro:property name="emissive" value="0 0 0 1"/>
   <xacro:arg name="simplified" default="false" />
   <xacro:macro name="grieel_gripper_first_finger_macro" params="prefix name *origin">
@@ -97,19 +93,4 @@
         </xacro:unless>
     </link>
-    <gazebo reference="${prefix}_${name}_phalanx1">
-        <material>Gazebo/Black</material>
-        <visual>
-            <material>
-                <ambient>${ambient}</ambient>
-                <diffuse>${diffuse}</diffuse>
-                <specular>${specular}</specular>
-                <emissive>${emissive}</emissive>
-            </material>
-        </visual>
-        <mu1>1.5</mu1>
-        <mu2>1.5</mu2>
-        <kp>1000000</kp>
-        <kd>1.0</kd>
-    </gazebo>
     <joint
         name="${prefix}_${name}_P12P2"
@@ -200,19 +181,4 @@
         </xacro:unless>
     </link>
-    <gazebo reference="${prefix}_${name}_phalanx2">
-        <material>Gazebo/Black</material>
-        <visual>
-            <material>
-                <ambient>${ambient}</ambient>
-                <diffuse>${diffuse}</diffuse>
-                <specular>${specular}</specular>
-                <emissive>${emissive}</emissive>
-            </material>
-        </visual>
-        <mu1>1.5</mu1>
-        <mu2>1.5</mu2>
-        <kp>1000000</kp>
-        <kd>1.0</kd>
-    </gazebo>
    <joint
         name="${prefix}_${name}_P22P3"
@@ -306,19 +272,4 @@
         </xacro:unless>
     </link>
-    <gazebo reference="${prefix}_${name}_phalanx3">
-        <material>Gazebo/Black</material>
-        <visual>
-            <material>
-                <ambient>${ambient}</ambient>
-                <diffuse>${diffuse}</diffuse>
-                <specular>${specular}</specular>
-                <emissive>${emissive}</emissive>
-            </material>
-        </visual>
-        <mu1>1.5</mu1>
-        <mu2>1.5</mu2>
-        <kp>1000000</kp>
-        <kd>1.0</kd>
-    </gazebo>
   </xacro:macro>
 </robot>

File: PARAM/lbr_description/urdf/Grieel/grieel_gazebo_colors.xacro (robot description, xacro)
@@ -8,8 +8,12 @@
         <xacro:include filename="$(find lbr_description)/urdf/Grieel/grieel_gripper_description.xacro" />
     </xacro:unless>
-    <xacro:property name="ambient" value="0.2 0.2 0.2 1"/>
-    <xacro:property name="diffuse" value="0.35 0.35 0.35 1"/>
-    <xacro:property name="specular" value="0.4 0.4 0.4 1"/>
-    <xacro:property name="emissive" value="0 0 0 1"/>
+    <xacro:property name="ambient" value="0.3 0.3 0.3 1"/>
+    <xacro:property name="diffuse" value="0.45 0.45 0.45 1"/>
+    <xacro:property name="specular" value="0.5 0.5 0.5 1"/>
+    <xacro:property name="emissive" value="0.001 0.001 0.001 1"/>
+    <xacro:property name="mu1" value="1.5"/>
+    <xacro:property name="mu2" value="1.5"/>
+    <xacro:property name="kp" value="1000000.0"/>
+    <xacro:property name="kd" value="1.0"/>
     <xacro:macro name="gazebo_colors_macro" params="prefix">
         <!-- Gazebo tag for support gripper/wheel phisical characteristics -->
@@ -30,14 +34,29 @@
             </gazebo>
         </xacro:unless> -->
-        <gazebo reference="${prefix}_femur">
-          <material>Gazebo/Black</material>
-            <visual>
-              <material>
-                <ambient>${ambient}</ambient>
-                <diffuse>${diffuse}</diffuse>
-                <specular>${specular}</specular>
-                <emissive>${emissive}</emissive>
-              </material>
-            </visual>
+          <gazebo reference="base_link">
+            <material>Gazebo/Black</material>
+            <visual>
+              <material>
+                  <ambient>${ambient}</ambient>
+                  <diffuse>${diffuse}</diffuse>
+                  <specular>${specular}</specular>
+                  <emissive>${emissive}</emissive>
+              </material>
+            </visual>
+            <mu1>${mu1}</mu1>
+            <mu2>${mu2}</mu2>
+            <kp>${kp}</kp>
+            <kd>${kd}</kd>
+          </gazebo>
+          <gazebo reference="${prefix}_femur">
+            <material>Gazebo/Black</material>
+              <visual>
+                <material>
+                  <ambient>${ambient}</ambient>
+                  <diffuse>${diffuse}</diffuse>
+                  <specular>${specular}</specular>
+                  <emissive>${emissive}</emissive>
+                </material>
+              </visual>
           </gazebo>
           <gazebo reference="${prefix}_tibia">
@@ -150,8 +169,368 @@
               </material>
             </visual>
-            <mu1>1.0</mu1>
-            <mu2>1.0</mu2>
-            <kp>1000000</kp>
-            <kd>1.0</kd>
+            <mu1>${mu1}</mu1>
+            <mu2>${mu2}</mu2>
+            <kp>${kp}</kp>
+            <kd>${kd}</kd>
+          </gazebo>
+          <gazebo reference="${prefix}_F1_phalanx1">
+              <material>Gazebo/Black</material>
+              <visual>
+                  <material>
+                      <ambient>${ambient}</ambient>
+                      <diffuse>${diffuse}</diffuse>
+                      <specular>${specular}</specular>
+                      <emissive>${emissive}</emissive>
+                  </material>
+              </visual>
+              <mu1>${mu1}</mu1>
+              <mu2>${mu2}</mu2>
+              <kp>${kp}</kp>
+              <kd>${kd}</kd>
+          </gazebo>
+          <gazebo reference="${prefix}_F1_phalanx2">
+              <material>Gazebo/Black</material>
+              <visual>
+                  <material>
+                      <ambient>${ambient}</ambient>
+                      <diffuse>${diffuse}</diffuse>
+                      <specular>${specular}</specular>
+                      <emissive>${emissive}</emissive>
+                  </material>
+              </visual>
+              <mu1>${mu1}</mu1>
+              <mu2>${mu2}</mu2>
+              <kp>${kp}</kp>
+              <kd>${kd}</kd>
+          </gazebo>
+          <gazebo reference="${prefix}_F1_phalanx3">
+              <material>Gazebo/Black</material>
+              <visual>
+                  <material>
+                      <ambient>${ambient}</ambient>
+                      <diffuse>${diffuse}</diffuse>
+                      <specular>${specular}</specular>
+                      <emissive>${emissive}</emissive>
+                  </material>
+              </visual>
+              <mu1>${mu1}</mu1>
+              <mu2>${mu2}</mu2>
+              <kp>${kp}</kp>
+              <kd>${kd}</kd>
+          </gazebo>
+          <gazebo reference="${prefix}_F2_phalanx1">
+              <material>Gazebo/Black</material>
+              <visual>
+                  <material>
+                      <ambient>${ambient}</ambient>
+                      <diffuse>${diffuse}</diffuse>
+                      <specular>${specular}</specular>
+                      <emissive>${emissive}</emissive>
+                  </material>
+              </visual>
+              <mu1>${mu1}</mu1>
+              <mu2>${mu2}</mu2>
+              <kp>${kp}</kp>
+              <kd>${kd}</kd>
+          </gazebo>
+          <gazebo reference="${prefix}_F2_phalanx2">
+              <material>Gazebo/Black</material>
+              <visual>
+                  <material>
+                      <ambient>${ambient}</ambient>
+                      <diffuse>${diffuse}</diffuse>
+                      <specular>${specular}</specular>
+                      <emissive>${emissive}</emissive>
+                  </material>
+              </visual>
+              <mu1>${mu1}</mu1>
+              <mu2>${mu2}</mu2>
+              <kp>${kp}</kp>
+              <kd>${kd}</kd>
+          </gazebo>
+          <gazebo reference="${prefix}_F2_phalanx3">
+              <material>Gazebo/Black</material>
+              <visual>
+                  <material>
+                      <ambient>${ambient}</ambient>
+                      <diffuse>${diffuse}</diffuse>
+                      <specular>${specular}</specular>
+                      <emissive>${emissive}</emissive>
+                  </material>
+              </visual>
+              <mu1>${mu1}</mu1>
+              <mu2>${mu2}</mu2>
+              <kp>${kp}</kp>
+              <kd>${kd}</kd>
+          </gazebo>
+          <gazebo reference="${prefix}_F3_phalanx1">
+              <material>Gazebo/Black</material>
+              <visual>
+                  <material>
+                      <ambient>${ambient}</ambient>
+                      <diffuse>${diffuse}</diffuse>
+                      <specular>${specular}</specular>
+                      <emissive>${emissive}</emissive>
+                  </material>
+              </visual>
+              <mu1>${mu1}</mu1>
+              <mu2>${mu2}</mu2>
+              <kp>${kp}</kp>
+              <kd>${kd}</kd>
+          </gazebo>
+          <gazebo reference="${prefix}_F3_phalanx2">
+              <material>Gazebo/Black</material>
+              <visual>
+                  <material>
+                      <ambient>${ambient}</ambient>
+                      <diffuse>${diffuse}</diffuse>
+                      <specular>${specular}</specular>
+                      <emissive>${emissive}</emissive>
+                  </material>
+              </visual>
+              <mu1>${mu1}</mu1>
+              <mu2>${mu2}</mu2>
+              <kp>${kp}</kp>
+              <kd>${kd}</kd>
+          </gazebo>
+          <gazebo reference="${prefix}_F3_phalanx3">
+              <material>Gazebo/Black</material>
+              <visual>
+                  <material>
+                      <ambient>${ambient}</ambient>
+                      <diffuse>${diffuse}</diffuse>
+                      <specular>${specular}</specular>
+                      <emissive>${emissive}</emissive>
+                  </material>
+              </visual>
+              <mu1>${mu1}</mu1>
+              <mu2>${mu2}</mu2>
+              <kp>${kp}</kp>
+              <kd>${kd}</kd>
+          </gazebo>
+          <gazebo reference="${prefix}_F4_phalanx1">
+              <material>Gazebo/Black</material>
+              <visual>
+                  <material>
+                      <ambient>${ambient}</ambient>
+                      <diffuse>${diffuse}</diffuse>
+                      <specular>${specular}</specular>
+                      <emissive>${emissive}</emissive>
+                  </material>
+              </visual>
+              <mu1>${mu1}</mu1>
+              <mu2>${mu2}</mu2>
+              <kp>${kp}</kp>
+              <kd>${kd}</kd>
+          </gazebo>
+          <gazebo reference="${prefix}_F4_phalanx2">
+              <material>Gazebo/Black</material>
+              <visual>
+                  <material>
+                      <ambient>${ambient}</ambient>
+                      <diffuse>${diffuse}</diffuse>
+                      <specular>${specular}</specular>
+                      <emissive>${emissive}</emissive>
+                  </material>
+              </visual>
+              <mu1>${mu1}</mu1>
+              <mu2>${mu2}</mu2>
+              <kp>${kp}</kp>
+              <kd>${kd}</kd>
+          </gazebo>
+          <gazebo reference="${prefix}_F4_phalanx3">
+              <material>Gazebo/Black</material>
+              <visual>
+                  <material>
+                      <ambient>${ambient}</ambient>
+                      <diffuse>${diffuse}</diffuse>
+                      <specular>${specular}</specular>
+                      <emissive>${emissive}</emissive>
+                  </material>
+              </visual>
+              <mu1>${mu1}</mu1>
+              <mu2>${mu2}</mu2>
+              <kp>${kp}</kp>
+              <kd>${kd}</kd>
+          </gazebo>
+          <gazebo reference="${prefix}_F5_phalanx1">
+              <material>Gazebo/Black</material>
+              <visual>
+                  <material>
+                      <ambient>${ambient}</ambient>
+                      <diffuse>${diffuse}</diffuse>
+                      <specular>${specular}</specular>
+                      <emissive>${emissive}</emissive>
+                  </material>
+              </visual>
+              <mu1>${mu1}</mu1>
+              <mu2>${mu2}</mu2>
+              <kp>${kp}</kp>
+              <kd>${kd}</kd>
+          </gazebo>
+          <gazebo reference="${prefix}_F5_phalanx2">
+              <material>Gazebo/Black</material>
+              <visual>
+                  <material>
+                      <ambient>${ambient}</ambient>
+                      <diffuse>${diffuse}</diffuse>
+                      <specular>${specular}</specular>
+                      <emissive>${emissive}</emissive>
+                  </material>
+              </visual>
+              <mu1>${mu1}</mu1>
+              <mu2>${mu2}</mu2>
+              <kp>${kp}</kp>
+              <kd>${kd}</kd>
+          </gazebo>
+          <gazebo reference="${prefix}_F5_phalanx3">
+              <material>Gazebo/Black</material>
+              <visual>
+                  <material>
+                      <ambient>${ambient}</ambient>
+                      <diffuse>${diffuse}</diffuse>
+                      <specular>${specular}</specular>
+                      <emissive>${emissive}</emissive>
+                  </material>
+              </visual>
+              <mu1>${mu1}</mu1>
+              <mu2>${mu2}</mu2>
+              <kp>${kp}</kp>
+              <kd>${kd}</kd>
+          </gazebo>
+          <gazebo reference="${prefix}_F6_phalanx1">
+              <material>Gazebo/Black</material>
+              <visual>
+                  <material>
+                      <ambient>${ambient}</ambient>
+                      <diffuse>${diffuse}</diffuse>
+                      <specular>${specular}</specular>
+                      <emissive>${emissive}</emissive>
+                  </material>
+              </visual>
+              <mu1>${mu1}</mu1>
+              <mu2>${mu2}</mu2>
+              <kp>${kp}</kp>
+              <kd>${kd}</kd>
+          </gazebo>
+          <gazebo reference="${prefix}_F6_phalanx2">
+              <material>Gazebo/Black</material>
+              <visual>
+                  <material>
+                      <ambient>${ambient}</ambient>
+                      <diffuse>${diffuse}</diffuse>
+                      <specular>${specular}</specular>
+                      <emissive>${emissive}</emissive>
+                  </material>
+              </visual>
+              <mu1>${mu1}</mu1>
+              <mu2>${mu2}</mu2>
+              <kp>${kp}</kp>
+              <kd>${kd}</kd>
+          </gazebo>
+          <gazebo reference="${prefix}_F6_phalanx3">
+              <material>Gazebo/Black</material>
+              <visual>
+                  <material>
+                      <ambient>${ambient}</ambient>
+                      <diffuse>${diffuse}</diffuse>
+                      <specular>${specular}</specular>
+                      <emissive>${emissive}</emissive>
+                  </material>
+              </visual>
+              <mu1>${mu1}</mu1>
+              <mu2>${mu2}</mu2>
+              <kp>${kp}</kp>
+              <kd>${kd}</kd>
+          </gazebo>
+          <gazebo reference="${prefix}_F7_phalanx1">
+              <material>Gazebo/Black</material>
+              <visual>
+                  <material>
+                      <ambient>${ambient}</ambient>
+                      <diffuse>${diffuse}</diffuse>
+                      <specular>${specular}</specular>
+                      <emissive>${emissive}</emissive>
+                  </material>
+              </visual>
+              <mu1>${mu1}</mu1>
+              <mu2>${mu2}</mu2>
+              <kp>${kp}</kp>
+              <kd>${kd}</kd>
+          </gazebo>
+          <gazebo reference="${prefix}_F7_phalanx2">
+              <material>Gazebo/Black</material>
+              <visual>
+                  <material>
+                      <ambient>${ambient}</ambient>
+                      <diffuse>${diffuse}</diffuse>
+                      <specular>${specular}</specular>
+                      <emissive>${emissive}</emissive>
+                  </material>
+              </visual>
+              <mu1>${mu1}</mu1>
+              <mu2>${mu2}</mu2>
+              <kp>${kp}</kp>
+              <kd>${kd}</kd>
+          </gazebo>
+          <gazebo reference="${prefix}_F7_phalanx3">
+              <material>Gazebo/Black</material>
+              <visual>
+                  <material>
+                      <ambient>${ambient}</ambient>
+                      <diffuse>${diffuse}</diffuse>
+                      <specular>${specular}</specular>
+                      <emissive>${emissive}</emissive>
+                  </material>
+              </visual>
+              <mu1>${mu1}</mu1>
+              <mu2>${mu2}</mu2>
+              <kp>${kp}</kp>
+              <kd>${kd}</kd>
+          </gazebo>
+          <gazebo reference="${prefix}_F8_phalanx1">
+              <material>Gazebo/Black</material>
+              <visual>
+                  <material>
+                      <ambient>${ambient}</ambient>
+                      <diffuse>${diffuse}</diffuse>
+                      <specular>${specular}</specular>
+                      <emissive>${emissive}</emissive>
+                  </material>
+              </visual>
+              <mu1>${mu1}</mu1>
+              <mu2>${mu2}</mu2>
+              <kp>${kp}</kp>
+              <kd>${kd}</kd>
+          </gazebo>
+          <gazebo reference="${prefix}_F8_phalanx2">
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
File: PARAM/lbr_description/urdf/Grieel/grieel_gripper_description.xacro (robot description, xacro)
@@ -8,6 +8,6 @@
     <xacro:include filename="$(find lbr_description)/urdf/Grieel/grieel_gripper_splitted.xacro" />
     <xacro:include filename="$(find lbr_description)/urdf/Grieel/inertial_macro.xacro" />
-    <xacro:property name="friction" value="0.4"/>
-    <xacro:property name="damping" value="0.15"/>
+    <xacro:property name="friction" value="0.5"/>
+    <xacro:property name="damping" value="0.2"/>
     <xacro:arg name="simplified" default="false" />
     <joint

File: PARAM/lbr_description/urdf/Grieel/lbr_base_description.xacro (robot description, xacro)
@@ -7,8 +7,8 @@
   <xacro:macro name="base_macro">
   <xacro:include filename="$(find lbr_description)/urdf/Grieel/inertial_macro.xacro" />
-  <xacro:property name="ambient" value="0.2 0.2 0.2 1"/>
-  <xacro:property name="diffuse" value="0.35 0.35 0.35 1"/>
-  <xacro:property name="specular" value="0.4 0.4 0.4 1"/>
-  <xacro:property name="emissive" value="0 0 0 1"/>
+    <xacro:property name="ambient" value="0.3 0.3 0.3 1"/>
+    <xacro:property name="diffuse" value="0.45 0.45 0.45 1"/>
+    <xacro:property name="specular" value="0.4 0.4 0.4 1"/>
+    <xacro:property name="emissive" value="0 0 0 1"/>
   <xacro:arg name="simplified" default="false" />
     <link
@@ -80,19 +80,4 @@
       </xacro:unless>
     </link>
-    <gazebo reference="base_link">
-      <material>Gazebo/Black</material>
-      <visual>
-        <material>
-            <ambient>${ambient}</ambient>
-            <diffuse>${diffuse}</diffuse>
-            <specular>${specular}</specular>
-            <emissive>${emissive}</emissive>
-        </material>
-      </visual>
-      <mu1>1.0</mu1>
-      <mu2>1.0</mu2>
-      <kp>1000000</kp>
-      <kd>1.0</kd>
-    </gazebo>
 <!--
     <link name="base_frame"/>

File: PARAM/lbr_description/urdf/Grieel/lbr_limb_description.xacro (robot description, xacro)
@@ -7,6 +7,6 @@
   <xacro:macro name="limb_macro" params="prefix parent radius">
     <xacro:include filename="$(find lbr_description)/urdf/Grieel/inertial_macro.xacro" />
-    <xacro:property name="friction" value="0.4"/>
-    <xacro:property name="damping" value="0.15"/>
+    <xacro:property name="friction" value="0.5"/>
+    <xacro:property name="damping" value="0.2"/>
     <xacro:arg name="simplified" default="false" />
     <joint
