Commit message: minor description changes

File: PARAM/lbr_description/urdf/Grieel/lbr_ros2_control.xacro (robot description, xacro)
@@ -28,9 +28,9 @@
         <state_interface name="velocity"/>
         <state_interface name="effort"/>
-        <!-- <transmission name="${prefix}_B2C_transmission">
+        <transmission name="${prefix}_B2C_transmission">
           <plugin>transmission_interface/SimpleTransmission</plugin>
           <param name="joint_to_actuator">272.5</param>
           <hardwareInterface>EffortJointInterface</hardwareInterface>
-        </transmission> -->
+        </transmission>
       </joint>
       <joint name="${prefix}_C2F">
@@ -56,9 +56,9 @@
         <state_interface name="velocity"/>
         <state_interface name="effort"/>
-        <!-- <transmission name="${prefix}_C2F_transmission">
+        <transmission name="${prefix}_C2F_transmission">
           <plugin>transmission_interface/SimpleTransmission</plugin>
           <param name="joint_to_actuator">272.5</param>
           <hardwareInterface>EffortJointInterface</hardwareInterface>
-        </transmission> -->
+        </transmission>
       </joint>
       <joint name="${prefix}_F2T">
@@ -84,9 +84,9 @@
         <state_interface name="velocity"/>
         <state_interface name="effort"/>
-        <!-- <transmission name="${prefix}_F2T_transmission">
+        <transmission name="${prefix}_F2T_transmission">
           <plugin>transmission_interface/SimpleTransmission</plugin>
           <param name="joint_to_actuator">353.5</param>
           <hardwareInterface>EffortJointInterface</hardwareInterface>
-        </transmission> -->
+        </transmission>
       </joint>
       <joint name="${prefix}_T2E">
@@ -112,9 +112,9 @@
         <state_interface name="velocity"/>
         <state_interface name="effort"/>
-        <!-- <transmission name="${prefix}_T2E_transmission">
+        <transmission name="${prefix}_T2E_transmission">
           <plugin>transmission_interface/SimpleTransmission</plugin>
           <param name="joint_to_actuator">353.5</param>
           <hardwareInterface>EffortJointInterface</hardwareInterface>
-        </transmission> -->
+        </transmission>
       </joint>
       <joint name="${prefix}_wristH">
@@ -145,9 +145,9 @@
         <state_interface name="velocity"/>
         <state_interface name="effort"/>
-        <!-- <transmission name="${prefix}_wristH_transmission">
+        <transmission name="${prefix}_wristH_transmission">
           <plugin>transmission_interface/SimpleTransmission</plugin>
           <param name="joint_to_actuator">257.4</param>
           <hardwareInterface>EffortJointInterface</hardwareInterface>
-        </transmission> -->
+        </transmission>
       </joint>
       <joint name="${prefix}_wristV">
@@ -178,9 +178,9 @@
         <state_interface name="velocity"/>
         <state_interface name="effort"/>
-        <!-- <transmission name="${prefix}_wristV_transmission">
+        <transmission name="${prefix}_wristV_transmission">
           <plugin>transmission_interface/SimpleTransmission</plugin>
           <param name="joint_to_actuator">257.4</param>
           <hardwareInterface>EffortJointInterface</hardwareInterface>
-        </transmission> -->
+        </transmission>
       </joint>
       <joint name="${prefix}_driving">
@@ -211,9 +211,9 @@
         <state_interface name="velocity"/>
         <state_interface name="effort"/>
-        <!-- <transmission name="${prefix}_driving_transmission">
+        <transmission name="${prefix}_driving_transmission">
           <plugin>transmission_interface/SimpleTransmission</plugin>
           <param name="joint_to_actuator">353.4</param>
           <hardwareInterface>EffortJointInterface</hardwareInterface>
-        </transmission> -->
+        </transmission>
       </joint>
     </ros2_control>
