Commit message: bug fixed and empty world

File: PARAM/lbr_description/urdf/Grieel/grieel_gazebo_colors.xacro (robot description, xacro)
@@ -35,6 +35,6 @@
         </xacro:unless> -->
           <gazebo reference="base_link">
-            <material>Gazebo/Black</material>
-            <visual>
+            <material>Gazebo/DarkGrey</material>
+            <!-- <visual>
               <material>
                   <ambient>${ambient}</ambient>
@@ -43,5 +43,5 @@
                   <emissive>${emissive}</emissive>
               </material>
-            </visual>
+            </visual> -->
             <mu1>${mu1}</mu1>
             <mu2>${mu2}</mu2>
@@ -50,5 +50,5 @@
           </gazebo>
           <gazebo reference="${prefix}_femur">
-            <material>Gazebo/Black</material>
+            <material>Gazebo/DarkGrey</material>
               <visual>
                 <material>
@@ -61,5 +61,5 @@
           </gazebo>
           <gazebo reference="${prefix}_tibia">
-            <material>Gazebo/Black</material>
+            <material>Gazebo/DarkGrey</material>
             <visual>
               <material>
@@ -72,5 +72,5 @@
           </gazebo>
           <gazebo reference="${prefix}_limb_end">
-            <material>Gazebo/Black</material>
+            <material>Gazebo/DarkGrey</material>
             <visual>
               <material>
@@ -83,5 +83,5 @@
           </gazebo>
           <gazebo reference="${prefix}_limb_root">
-            <material>Gazebo/Black</material>
+            <material>Gazebo/DarkGrey</material>
             <visual>
               <material>
@@ -94,5 +94,5 @@
           </gazebo>
           <gazebo reference="${prefix}_coxa">
-            <material>Gazebo/Black</material>
+            <material>Gazebo/DarkGrey</material>
             <visual>
               <material>
@@ -105,5 +105,5 @@
           </gazebo>
           <gazebo reference="${prefix}_wristH_Link">
-            <material>Gazebo/Black</material>
+            <material>Gazebo/DarkGrey</material>
             <visual>
               <material>
@@ -116,5 +116,5 @@
           </gazebo>
           <gazebo reference="${prefix}_wristV_Link">
-            <material>Gazebo/Black</material>
+            <material>Gazebo/DarkGrey</material>
             <visual>
               <material>
@@ -127,5 +127,5 @@
           </gazebo>
           <gazebo reference="${prefix}_driving_Link">
-            <material>Gazebo/Black</material>
+            <material>Gazebo/DarkGrey</material>
             <visual>
               <material>
@@ -138,5 +138,5 @@
           </gazebo>
           <!-- <gazebo reference="${prefix}_gripper_Link">
-            <material>Gazebo/Black</material>
+            <material>Gazebo/DarkGrey</material>
             <visual>
               <material>
@@ -149,5 +149,5 @@
           </gazebo>
           <gazebo reference="${prefix}_wheel_Link">
-            <material>Gazebo/Black</material>
+            <material>Gazebo/DarkGrey</material>
             <visual>
               <material>
@@ -160,5 +160,5 @@
           </gazebo> -->
           <gazebo reference="${prefix}_hand_Link">
-            <material>Gazebo/Black</material>
+            <material>Gazebo/DarkGrey</material>
             <visual>
               <material>
@@ -175,5 +175,5 @@
           </gazebo>
           <gazebo reference="${prefix}_F1_phalanx1">
-              <material>Gazebo/Black</material>
+              <material>Gazebo/DarkGrey</material>
               <visual>
                   <material>
@@ -190,5 +190,5 @@
           </gazebo>
           <gazebo reference="${prefix}_F1_phalanx2">
-              <material>Gazebo/Black</material>
+              <material>Gazebo/DarkGrey</material>
               <visual>
                   <material>
@@ -205,5 +205,5 @@
           </gazebo>
           <gazebo reference="${prefix}_F1_phalanx3">
-              <material>Gazebo/Black</material>
+              <material>Gazebo/DarkGrey</material>
               <visual>
                   <material>
@@ -220,5 +220,5 @@
           </gazebo>
           <gazebo reference="${prefix}_F2_phalanx1">
-              <material>Gazebo/Black</material>
+              <material>Gazebo/DarkGrey</material>
               <visual>
                   <material>
@@ -235,5 +235,5 @@
           </gazebo>
           <gazebo reference="${prefix}_F2_phalanx2">
-              <material>Gazebo/Black</material>
+              <material>Gazebo/DarkGrey</material>
               <visual>
                   <material>
@@ -250,5 +250,5 @@
           </gazebo>
           <gazebo reference="${prefix}_F2_phalanx3">
-              <material>Gazebo/Black</material>
+              <material>Gazebo/DarkGrey</material>
               <visual>
                   <material>
@@ -265,5 +265,5 @@
           </gazebo>
           <gazebo reference="${prefix}_F3_phalanx1">
-              <material>Gazebo/Black</material>
+              <material>Gazebo/DarkGrey</material>
               <visual>
                   <material>
@@ -280,5 +280,5 @@
           </gazebo>
           <gazebo reference="${prefix}_F3_phalanx2">
-              <material>Gazebo/Black</material>
+              <material>Gazebo/DarkGrey</material>
               <visual>
                   <material>
@@ -295,5 +295,5 @@
           </gazebo>
           <gazebo reference="${prefix}_F3_phalanx3">
-              <material>Gazebo/Black</material>
+              <material>Gazebo/DarkGrey</material>
               <visual>
                   <material>
@@ -310,5 +310,5 @@
           </gazebo>
           <gazebo reference="${prefix}_F4_phalanx1">
-              <material>Gazebo/Black</material>
+              <material>Gazebo/DarkGrey</material>
               <visual>
                   <material>
@@ -325,5 +325,5 @@
           </gazebo>
           <gazebo reference="${prefix}_F4_phalanx2">
-              <material>Gazebo/Black</material>
+              <material>Gazebo/DarkGrey</material>
               <visual>
                   <material>
@@ -340,5 +340,5 @@
           </gazebo>
           <gazebo reference="${prefix}_F4_phalanx3">
-              <material>Gazebo/Black</material>
+              <material>Gazebo/DarkGrey</material>
               <visual>
                   <material>
@@ -355,5 +355,5 @@
           </gazebo>
           <gazebo reference="${prefix}_F5_phalanx1">
-              <material>Gazebo/Black</material>
+              <material>Gazebo/DarkGrey</material>
               <visual>
                   <material>
@@ -370,5 +370,5 @@
           </gazebo>
           <gazebo reference="${prefix}_F5_phalanx2">
-              <material>Gazebo/Black</material>
+              <material>Gazebo/DarkGrey</material>
               <visual>
                   <material>
@@ -385,5 +385,5 @@
           </gazebo>
           <gazebo reference="${prefix}_F5_phalanx3">
-              <material>Gazebo/Black</material>
+              <material>Gazebo/DarkGrey</material>
               <visual>
                   <material>
@@ -400,5 +400,5 @@
           </gazebo>
           <gazebo reference="${prefix}_F6_phalanx1">
-              <material>Gazebo/Black</material>
+              <material>Gazebo/DarkGrey</material>
               <visual>
                   <material>
@@ -415,5 +415,5 @@
           </gazebo>
           <gazebo reference="${prefix}_F6_phalanx2">
-              <material>Gazebo/Black</material>
+              <material>Gazebo/DarkGrey</material>
               <visual>
                   <material>
@@ -430,5 +430,5 @@
           </gazebo>
           <gazebo reference="${prefix}_F6_phalanx3">
-              <material>Gazebo/Black</material>
+              <material>Gazebo/DarkGrey</material>
               <visual>
                   <material>
@@ -445,5 +445,5 @@
           </gazebo>
           <gazebo reference="${prefix}_F7_phalanx1">
-              <material>Gazebo/Black</material>
+              <material>Gazebo/DarkGrey</material>
               <visual>
                   <material>
@@ -460,5 +460,5 @@
           </gazebo>
           <gazebo reference="${prefix}_F7_phalanx2">
-              <material>Gazebo/Black</material>
+              <material>Gazebo/DarkGrey</material>
               <visual>
                   <material>
@@ -475,5 +475,5 @@
           </gazebo>
           <gazebo reference="${prefix}_F7_phalanx3">
-              <material>Gazebo/Black</material>
+              <material>Gazebo/DarkGrey</material>
               <visual>
                   <material>
@@ -490,5 +490,5 @@
           </gazebo>
           <gazebo reference="${prefix}_F8_phalanx1">
-              <material>Gazebo/Black</material>
+              <material>Gazebo/DarkGrey</material>
               <visual>
                   <material>
@@ -505,5 +505,5 @@
           </gazebo>
           <gazebo reference="${prefix}_F8_phalanx2">
-              <material>Gazebo/Black</material>
+              <material>Gazebo/DarkGrey</material>
               <visual>
                   <material>
@@ -520,5 +520,5 @@
           </gazebo>
           <gazebo reference="${prefix}_F8_phalanx3">
-              <material>Gazebo/Black</material>
+              <material>Gazebo/DarkGrey</material>
               <visual>
                   <material>
